Commit message: Upgraded

File: demo_navi/src/urdf/model.urdf.xacro (robot description, xacro)
@@ -8,13 +8,12 @@
   <link name="base_link">
     <inertial>
-      <origin rpy="0 0 0" xyz="-0.15 0 0.045"/>
-      <mass value="0.07862944645"/>
-      <inertia ixx="0.00002035985530754" ixy="0" ixz="0" iyy="0.00002035985530754" iyz="0" izz="0.00003945961663220"/>
-    </inertial>
-    <visual>
-      <origin rpy="-1.57 0 1.57" xyz="0.075 -0.325 0.112"/>
+      <origin rpy="0 0 0" xyz="-0.147 0 0"/>
+      <mass value="5"/>
+      <inertia ixx="0.15" ixy="0" ixz="0" iyy="0.104167" iyz="0" izz="0.254167"/>
+    </inertial>
+    <visual>
+      <origin rpy="0 0 0" xyz="0 0 0"/>
       <geometry>
         <mesh filename="package://demo_navi/src/meshes/base_link.stl"/>
-        <scale>0.001 0.001 0.001</scale>
       </geometry>
       <material name="base_material">
@@ -23,5 +22,5 @@
     </visual>
     <collision>
-      <origin rpy="-1.57 0 1.57" xyz="0.075 -0.325 0.112"/>
+      <origin rpy="0 0 0" xyz="0 0 0"/>
       <geometry>
         <mesh filename="package://demo_navi/src/meshes/base_link.stl"/>
@@ -32,11 +31,11 @@
     <parent link="base_footprint"/>
     <child link="base_link"/>
-    <origin xyz="0 0 0.01905"/>
+    <origin xyz="0 0 0"/>
   </joint>
   <link name="rim_left_link">
     <inertial>
       <origin xyz="0 0 0"/>
-      <mass value="0.0083578"/>
-      <inertia ixx="2.75e-07" ixy="0" ixz="0" iyy="2.75e-07" iyz="0" izz="3.43e-07"/>
+      <mass value="1"/>
+      <inertia ixx="0.0007" ixy="0" ixz="0" iyy="0.0007" iyz="0" izz="0.0008"/>
     </inertial>
     <visual>
@@ -52,12 +51,4 @@
         <mesh filename="package://demo_navi/src/meshes/rim.stl"/>
       </geometry>
-      <surface>
-        <friction>
-          <ode>
-            <mu>0.1</mu>
-            <mu2>0.1</mu2>
-          </ode>
-        </friction>
-      </surface>
     </collision>
   </link>
@@ -65,34 +56,26 @@
     <parent link="base_link"/>
     <child link="rim_left_link"/>
-    <axis xyz="0 0 1"/>
-    <origin rpy="1.570796326794896 0 -0.523599" xyz="-0.03 0.215 0.04"/>
-    <limit effort="100000" velocity="100000"/>
-    <joint_properties friction="1.0"/>
+    <axis xyz="1 0 0"/>
+    <origin rpy="0 0 -2.0944" xyz="-0.0267 0.214 0.04"/>
+    <!--<limit effort="100000" velocity="100000"/>
+			<joint_properties friction="1.0"/>-->
   </joint>
   <link name="roller_s_rim_left_link">
     <inertial>
-      <mass value="0.0011"/>
-      <inertia ixx="2e-08" ixy="0" ixz="0" iyy="2e-08" iyz="0" izz="9e-08"/>
-    </inertial>
-    <visual>
-      <geometry>
-        <mesh filename="package://demo_navi/src/meshes/roller1.stl"/>
-      </geometry>
-      <material name="roller_material">
-        <color rgba="0.1 0.1 0.1 1"/>
-      </material>
-    </visual>
-    <collision>
-      <geometry>
-        <mesh filename="package://demo_navi/src/meshes/roller1.stl"/>
-      </geometry>
-      <surface>
-        <friction>
-          <ode>
-            <mu>0.1</mu>
-            <mu2>0.1</mu2>
-          </ode>
-        </friction>
-      </surface>
+      <mass value="0.1"/>
+      <inertia ixx="6.8e-05" ixy="0" ixz="0" iyy="6.8e-05" iyz="0" izz="0.000101"/>
+    </inertial>
+    <visual>
+      <geometry>
+        <mesh filename="package://demo_navi/src/meshes/roller.stl"/>
+      </geometry>
+      <material name="roller_material">
+        <color rgba="0.1 0.1 0.1 1"/>
+      </material>
+    </visual>
+    <collision>
+      <geometry>
+        <mesh filename="package://demo_navi/src/meshes/roller.stl"/>
+      </geometry>
     </collision>
   </link>
@@ -100,46 +83,37 @@
     <parent link="rim_left_link"/>
     <child link="roller_s_rim_left_link"/>
-    <axis xyz="1 0 0"/>
-    <origin rpy="0 0 3.1415" xyz="0 -0.025 0.014"/>
+    <axis xyz="0 1 0"/>
+    <origin rpy="0 0 0" xyz="0.0153 0 -0.0266"/>
   </joint>
   <gazebo reference="roller_s_rim_left_link">
-    <dampingFactor>10</dampingFactor>
-    <minDepth>0.001</minDepth>
-    <fdir1>0 0 1</fdir1>
-    <kp>500000.0</kp>
-    <kd>10.0</kd>
-    <maxVel>0.1</maxVel>
-    <fdir1>1 0 0</fdir1>
-    <material>Gazebo/Grey</material>
-  </gazebo>
-  <gazebo reference="roller_s_rim_left_joint">
-    <dampingFactor>10</dampingFactor>
-    <minDepth>0.001</minDepth>
-  </gazebo>
+    <!--<mu1>5000.0</mu1>
+  				<mu2>2500.0</mu2>
+      			<kp  value="10000000.0" />
+      			<maxContacts  value="10" />
+      			<kd  value="1.0" />
+      			<fdir1 value="1 0 0"/>-->
+    <material>Gazebo/Grey</material>
+  </gazebo>
+  <!--<gazebo reference="roller_${name}_rim_${parent}_joint">
+    <dampingFactor>10</dampingFactor>
+    <minDepth>0.001</minDepth>
+  </gazebo>-->
   <link name="roller_nw_rim_left_link">
     <inertial>
-      <mass value="0.0011"/>
-      <inertia ixx="2e-08" ixy="0" ixz="0" iyy="2e-08" iyz="0" izz="9e-08"/>
-    </inertial>
-    <visual>
-      <geometry>
-        <mesh filename="package://demo_navi/src/meshes/roller1.stl"/>
-      </geometry>
-      <material name="roller_material">
-        <color rgba="0.1 0.1 0.1 1"/>
-      </material>
-    </visual>
-    <collision>
-      <geometry>
-        <mesh filename="package://demo_navi/src/meshes/roller1.stl"/>
-      </geometry>
-      <surface>
-        <friction>
-          <ode>
-            <mu>0.1</mu>
-            <mu2>0.1</mu2>
-          </ode>
-        </friction>
-      </surface>
+      <mass value="0.1"/>
+      <inertia ixx="6.8e-05" ixy="0" ixz="0" iyy="6.8e-05" iyz="0" izz="0.000101"/>
+    </inertial>
+    <visual>
+      <geometry>
+        <mesh filename="package://demo_navi/src/meshes/roller.stl"/>
+      </geometry>
+      <material name="roller_material">
+        <color rgba="0.1 0.1 0.1 1"/>
+      </material>
+    </visual>
+    <collision>
+      <geometry>
+        <mesh filename="package://demo_navi/src/meshes/roller.stl"/>
+      </geometry>
     </collision>
   </link>
@@ -147,46 +121,37 @@
     <parent link="rim_left_link"/>
     <child link="roller_nw_rim_left_link"/>
-    <axis xyz="1 0 0"/>
-    <origin rpy="0 0 1.0472" xyz="-0.0215 0.0125 0.014"/>
+    <axis xyz="0 1 0"/>
+    <origin rpy="1.0472 0 0" xyz="0.015 -0.0231 0.0131"/>
   </joint>
   <gazebo reference="roller_nw_rim_left_link">
-    <dampingFactor>10</dampingFactor>
-    <minDepth>0.001</minDepth>
-    <fdir1>0 0 1</fdir1>
-    <kp>500000.0</kp>
-    <kd>10.0</kd>
-    <maxVel>0.1</maxVel>
-    <fdir1>1 0 0</fdir1>
-    <material>Gazebo/Grey</material>
-  </gazebo>
-  <gazebo reference="roller_nw_rim_left_joint">
-    <dampingFactor>10</dampingFactor>
-    <minDepth>0.001</minDepth>
-  </gazebo>
+    <!--<mu1>5000.0</mu1>
+  				<mu2>2500.0</mu2>
+      			<kp  value="10000000.0" />
+      			<maxContacts  value="10" />
+      			<kd  value="1.0" />
+      			<fdir1 value="1 0 0"/>-->
+    <material>Gazebo/Grey</material>
+  </gazebo>
+  <!--<gazebo reference="roller_${name}_rim_${parent}_joint">
+    <dampingFactor>10</dampingFactor>
+    <minDepth>0.001</minDepth>
+  </gazebo>-->
   <link name="roller_ne_rim_left_link">
     <inertial>
-      <mass value="0.0011"/>
-      <inertia ixx="2e-08" ixy="0" ixz="0" iyy="2e-08" iyz="0" izz="9e-08"/>
-    </inertial>
-    <visual>
-      <geometry>
-        <mesh filename="package://demo_navi/src/meshes/roller1.stl"/>
-      </geometry>
-      <material name="roller_material">
-        <color rgba="0.1 0.1 0.1 1"/>
-      </material>
-    </visual>
-    <collision>
-      <geometry>
-        <mesh filename="package://demo_navi/src/meshes/roller1.stl"/>
-      </geometry>
-      <surface>
-        <friction>
-          <ode>
-            <mu>0.1</mu>
-            <mu2>0.1</mu2>
-          </ode>
-        </friction>
-      </surface>
+      <mass value="0.1"/>
+      <inertia ixx="6.8e-05" ixy="0" ixz="0" iyy="6.8e-05" iyz="0" izz="0.000101"/>
+    </inertial>
+    <visual>
+      <geometry>
+        <mesh filename="package://demo_navi/src/meshes/roller.stl"/>
+      </geometry>
+      <material name="roller_material">
+        <color rgba="0.1 0.1 0.1 1"/>
+      </material>
+    </visual>
+    <collision>
+      <geometry>
+        <mesh filename="package://demo_navi/src/meshes/roller.stl"/>
+      </geometry>
     </collision>
   </link>
@@ -194,46 +159,37 @@
     <parent link="rim_left_link"/>
     <child link="roller_ne_rim_left_link"/>
-    <axis xyz="1 0 0"/>
-    <origin rpy="0 0 -1.0472" xyz="0.0215 0.0125 0.014"/>
+    <axis xyz="0 1 0"/>
+    <origin rpy="-1.0472 0 0" xyz="0.015 0.0231 0.0135"/>
   </joint>
   <gazebo reference="roller_ne_rim_left_link">
-    <dampingFactor>10</dampingFactor>
-    <minDepth>0.001</minDepth>
-    <fdir1>0 0 1</fdir1>
-    <kp>500000.0</kp>
-    <kd>10.0</kd>
-    <maxVel>0.1</maxVel>
-    <fdir1>1 0 0</fdir1>
-    <material>Gazebo/Grey</material>
-  </gazebo>
-  <gazebo reference="roller_ne_rim_left_joint">
-    <dampingFactor>10</dampingFactor>
-    <minDepth>0.001</minDepth>
-  </gazebo>
+    <!--<mu1>5000.0</mu1>
+  				<mu2>2500.0</mu2>
+      			<kp  value="10000000.0" />
+      			<maxContacts  value="10" />
+      			<kd  value="1.0" />
+      			<fdir1 value="1 0 0"/>-->
+    <material>Gazebo/Grey</material>
+  </gazebo>
+  <!--<gazebo reference="roller_${name}_rim_${parent}_joint">
+    <dampingFactor>10</dampingFactor>
+    <minDepth>0.001</minDepth>
+  </gazebo>-->
   <link name="roller_sw_rim_left_link">
     <inertial>
-      <mass value="0.0011"/>
-      <inertia ixx="2e-08" ixy="0" ixz="0" iyy="2e-08" iyz="0" izz="9e-08"/>
-    </inertial>
-    <visual>
-      <geometry>
-        <mesh filename="package://demo_navi/src/meshes/roller1.stl"/>
-      </geometry>
-      <material name="roller_material">
-        <color rgba="0.1 0.1 0.1 1"/>
-      </material>
-    </visual>
-    <collision>
-      <geometry>
-        <mesh filename="package://demo_navi/src/meshes/roller1.stl"/>
-      </geometry>
-      <surface>
-        <friction>
-          <ode>
-            <mu>0.1</mu>
-            <mu2>0.1</mu2>
-          </ode>
-        </friction>
-      </surface>
+      <mass value="0.1"/>
+      <inertia ixx="6.8e-05" ixy="0" ixz="0" iyy="6.8e-05" iyz="0" izz="0.000101"/>
+    </inertial>
+    <visual>
+      <geometry>
+        <mesh filename="package://demo_navi/src/meshes/roller.stl"/>
+      </geometry>
+      <material name="roller_material">
+        <color rgba="0.1 0.1 0.1 1"/>
+      </material>
+    </visual>
+    <collision>
+      <geometry>
+        <mesh filename="package://demo_navi/src/meshes/roller.stl"/>
+      </geometry>
     </collision>
   </link>
@@ -241,46 +197,37 @@
     <parent link="rim_left_link"/>
     <child link="roller_sw_rim_left_link"/>
-    <axis xyz="1 0 0"/>
-    <origin rpy="0 0 1.0472" xyz="0.0215 -0.0125 -0.014"/>
+    <axis xyz="0 1 0"/>
+    <origin rpy="1.0472 0 0" xyz="-0.0146 0.023 -0.0133"/>
   </joint>
   <gazebo reference="roller_sw_rim_left_link">
-    <dampingFactor>10</dampingFactor>
-    <minDepth>0.001</minDepth>
-    <fdir1>0 0 1</fdir1>
-    <kp>500000.0</kp>
-    <kd>10.0</kd>
-    <maxVel>0.1</maxVel>
-    <fdir1>1 0 0</fdir1>
-    <material>Gazebo/Grey</material>
-  </gazebo>
-  <gazebo reference="roller_sw_rim_left_joint">
-    <dampingFactor>10</dampingFactor>
-    <minDepth>0.001</minDepth>
-  </gazebo>
+    <!--<mu1>5000.0</mu1>
+  				<mu2>2500.0</mu2>
+      			<kp  value="10000000.0" />
+      			<maxContacts  value="10" />
+      			<kd  value="1.0" />
+      			<fdir1 value="1 0 0"/>-->
+    <material>Gazebo/Grey</material>
+  </gazebo>
+  <!--<gazebo reference="roller_${name}_rim_${parent}_joint">
+    <dampingFactor>10</dampingFactor>
+    <minDepth>0.001</minDepth>
+  </gazebo>-->
   <link name="roller_n_rim_left_link">
     <inertial>
-      <mass value="0.0011"/>
-      <inertia ixx="2e-08" ixy="0" ixz="0" iyy="2e-08" iyz="0" izz="9e-08"/>
-    </inertial>
-    <visual>
-      <geometry>
-        <mesh filename="package://demo_navi/src/meshes/roller1.stl"/>
-      </geometry>
-      <material name="roller_material">
-        <color rgba="0.1 0.1 0.1 1"/>
-      </material>
-    </visual>
-    <collision>
-      <geometry>
-        <mesh filename="package://demo_navi/src/meshes/roller1.stl"/>
-      </geometry>
-      <surface>
-        <friction>
-          <ode>
-            <mu>0.1</mu>
-            <mu2>0.1</mu2>
-          </ode>
-        </friction>
-      </surface>
+      <mass value="0.1"/>
+      <inertia ixx="6.8e-05" ixy="0" ixz="0" iyy="6.8e-05" iyz="0" izz="0.000101"/>
+    </inertial>
+    <visual>
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