Commit message: Updated

File: demo_navi/src/urdf/model.urdf.xacro (robot description, xacro)
@@ -921,4 +921,5 @@
   <link name="shoulder_link">
     <visual>
+      <origin rpy="0 0 0" xyz="0 0 0"/>
       <geometry>
         <mesh filename="package://demo_navi/src/meshes/arm/shoulder_link.stl"/>
@@ -929,4 +930,5 @@
     </visual>
     <collision>
+      <origin rpy="0 0 0" xyz="0 0 0"/>
       <geometry>
         <mesh filename="package://demo_navi/src/meshes/arm/shoulder_link.stl"/>
@@ -934,4 +936,5 @@
     </collision>
     <inertial>
+      <origin rpy="0 0 0" xyz="0 0 0"/>
       <mass value="0.1"/>
       <inertia ixx="0.1" ixy="0.0" ixz="0.0" iyy="0.1" iyz="0.0" izz="0.1"/>
@@ -940,4 +943,5 @@
   <link name="biceps_link">
     <visual>
+      <origin rpy="0 0 0" xyz="0.04825 0 0.14"/>
       <geometry>
         <mesh filename="package://demo_navi/src/meshes/arm/biceps_link.stl"/>
@@ -948,4 +952,5 @@
     </visual>
     <collision>
+      <origin rpy="0 0 0" xyz="0.04825 0 0.14"/>
       <geometry>
         <mesh filename="package://demo_navi/src/meshes/arm/biceps_link.stl"/>
@@ -953,4 +958,5 @@
     </collision>
     <inertial>
+      <origin rpy="0 0 0" xyz="0.04825 0 0.14"/>
       <mass value="0.1"/>
       <inertia ixx="0.1" ixy="0.0" ixz="0.0" iyy="0.1" iyz="0.0" izz="0.1"/>
@@ -959,4 +965,5 @@
   <link name="forearm_link">
     <visual>
+      <origin rpy="0 0 0" xyz="0 0 0.14203"/>
       <geometry>
         <mesh filename="package://demo_navi/src/meshes/arm/forearm_link.stl"/>
@@ -967,4 +974,5 @@
     </visual>
     <collision>
+      <origin rpy="0 0 0" xyz="0 0 0.14203"/>
       <geometry>
         <mesh filename="package://demo_navi/src/meshes/arm/forearm_link.stl"/>
@@ -972,4 +980,5 @@
     </collision>
     <inertial>
+      <origin rpy="0 0 0" xyz="0 0 0.14203"/>
       <mass value="0.1"/>
       <inertia ixx="1.0" ixy="0.0" ixz="0.0" iyy="1.0" iyz="0.0" izz="1.0"/>
@@ -978,4 +987,5 @@
   <link name="wrist_1_link">
     <visual>
+      <origin rpy="0 0 0" xyz="0 0 0"/>
       <geometry>
         <mesh filename="package://demo_navi/src/meshes/arm/wrist_1_link.stl"/>
@@ -986,4 +996,5 @@
     </visual>
     <collision>
+      <origin rpy="0 0 0" xyz="0 0 0"/>
       <geometry>
         <mesh filename="package://demo_navi/src/meshes/arm/wrist_1_link.stl"/>
@@ -991,4 +1002,5 @@
     </collision>
     <inertial>
+      <origin rpy="0 0 0" xyz="0 0 0"/>
       <mass value="0.1"/>
       <inertia ixx="0.1" ixy="0.0" ixz="0.0" iyy="0.1" iyz="0.0" izz="0.1"/>
@@ -997,4 +1009,5 @@
   <link name="wrist_2_link">
     <visual>
+      <origin rpy="0 0 0" xyz="0 0 0.043"/>
       <geometry>
         <mesh filename="package://demo_navi/src/meshes/arm/wrist_2_link.stl"/>
@@ -1005,4 +1018,5 @@
     </visual>
     <collision>
+      <origin rpy="0 0 0" xyz="0 0 0.043"/>
       <geometry>
         <mesh filename="package://demo_navi/src/meshes/arm/wrist_2_link.stl"/>
@@ -1010,4 +1024,5 @@
     </collision>
     <inertial>
+      <origin rpy="0 0 0" xyz="0 0 0.043"/>
       <mass value="0.1"/>
       <inertia ixx="0.1" ixy="0.0" ixz="0.0" iyy="0.1" iyz="0.0" izz="0.1"/>
@@ -1016,4 +1031,5 @@
   <link name="gripper_rail_link">
     <visual>
+      <origin rpy="0 0 1.57" xyz="0 0 0"/>
       <geometry>
         <mesh filename="package://demo_navi/src/meshes/arm/gripper_rail_link.stl"/>
@@ -1024,4 +1040,5 @@
     </visual>
     <collision>
+      <origin rpy="0 0 1.57" xyz="0 0 0"/>
       <geometry>
         <mesh filename="package://demo_navi/src/meshes/arm/gripper_rail_link.stl"/>
@@ -1029,10 +1046,14 @@
     </collision>
     <inertial>
+      <origin rpy="0 0 1.57" xyz="0 0 0"/>
       <mass value="0.1"/>
       <inertia ixx="0.1" ixy="0.0" ixz="0.0" iyy="0.1" iyz="0.0" izz="0.1"/>
     </inertial>
   </link>
+  <link name="gripper_aux_link">
+      </link>
   <link name="gripper_1_link">
     <visual>
+      <origin rpy="0 0 1.57" xyz="0 -0.0007 0"/>
       <geometry>
         <mesh filename="package://demo_navi/src/meshes/arm/gripper_hand_fixed_link.stl"/>
@@ -1043,4 +1064,5 @@
     </visual>
     <collision>
+      <origin rpy="0 0 1.57" xyz="0 -0.0007 0"/>
       <geometry>
         <mesh filename="package://demo_navi/src/meshes/arm/gripper_hand_fixed_link.stl"/>
@@ -1048,4 +1070,5 @@
     </collision>
     <inertial>
+      <origin rpy="0 0 1.57" xyz="0 -0.0007 0"/>
       <mass value="0.1"/>
       <inertia ixx="0.1" ixy="0.0" ixz="0.0" iyy="0.1" iyz="0.0" izz="0.1"/>
@@ -1054,4 +1077,5 @@
   <link name="gripper_2_link">
     <visual>
+      <origin rpy="0 0 -1.57" xyz="0 0.0007 0"/>
       <geometry>
         <mesh filename="package://demo_navi/src/meshes/arm/gripper_hand_fixed_link.stl"/>
@@ -1062,4 +1086,5 @@
     </visual>
     <collision>
+      <origin rpy="0 0 -1.57" xyz="0 0.0007 0"/>
       <geometry>
         <mesh filename="package://demo_navi/src/meshes/arm/gripper_hand_fixed_link.stl"/>
@@ -1067,4 +1092,5 @@
     </collision>
     <inertial>
+      <origin rpy="0 0 -1.57" xyz="0 0.0007 0"/>
       <mass value="0.1"/>
       <inertia ixx="0.1" ixy="0.0" ixz="0.0" iyy="0.1" iyz="0.0" izz="0.1"/>
@@ -1073,5 +1099,5 @@
   <!-- joints -->
   <joint name="joint_1" type="revolute">
-    <origin rpy="0 0 0" xyz="0.0033 -0.0017 0.15"/>
+    <origin rpy="0 0 0" xyz="0 0 0.15"/>
     <parent link="base_link"/>
     <child link="shoulder_link"/>
@@ -1081,5 +1107,5 @@
   <joint name="joint_2" type="revolute">
     <!--origin xyz="0.04825 0 0.14203" rpy="0 0 0" /-->
-    <origin rpy="0 0 0" xyz="0.051 0.003 0.142"/>
+    <origin rpy="0 0 0" xyz="0 0 0"/>
     <parent link="shoulder_link"/>
     <child link="biceps_link"/>
@@ -1088,5 +1114,5 @@
   </joint>
   <joint name="joint_3" type="revolute">
-    <origin rpy="0 0 0" xyz="-0.002 -0.003 0.14057"/>
+    <origin rpy="0 1.571 0" xyz="0.04825 0 0.14203"/>
     <parent link="biceps_link"/>
     <child link="forearm_link"/>
@@ -1095,5 +1121,5 @@
   </joint>
   <joint name="joint_4" type="revolute">
-    <origin rpy="0 0 0" xyz="0.0027 -0.002 0.008"/>
+    <origin rpy="0 0 0" xyz="0 0 0.14203"/>
     <parent link="forearm_link"/>
     <child link="wrist_1_link"/>
@@ -1102,5 +1128,5 @@
   </joint>
   <joint name="joint_5" type="revolute">
-    <origin rpy="0 0 0" xyz="0 0 0.08"/>
+    <origin rpy="0 0 0" xyz="0 0 0.0715"/>
     <parent link="wrist_1_link"/>
     <child link="wrist_2_link"/>
@@ -1108,6 +1134,6 @@
     <limit effort="0" lower="-2.617" upper="2.617" velocity="1.571"/>
   </joint>
-  <joint name="joint_6" type="revolute">
-    <origin rpy="0 0 0" xyz="0 0 0.04"/>
+  <joint name="joint_6" type="fixed">
+    <origin rpy="0 0 0" xyz="0 0 0.043"/>
     <parent link="wrist_2_link"/>
     <child link="gripper_rail_link"/>
@@ -1115,17 +1141,24 @@
     <limit effort="0" lower="-0.31" upper="0.1" velocity="0.5"/>
   </joint>
+  <joint name="gripper_revolute_joint" type="revolute">
+    <origin rpy="0 0 0" xyz="0 0 0"/>
+    <parent link="gripper_rail_link"/>
+    <child link="gripper_aux_link"/>
+    <axis xyz="0 0 1"/>
+    <limit effort="0" lower="0" upper="2.6" velocity="0.5"/>
+  </joint>
   <joint name="gripper_prismatic_joint_1" type="prismatic">
     <origin rpy="0 0 0" xyz="0 0 0"/>
     <parent link="gripper_rail_link"/>
     <child link="gripper_1_link"/>
-    <axis xyz="0 1 0"/>
+    <axis xyz="0 -1 0"/>
     <limit effort="0" lower="0" upper="0.027" velocity="0.5"/>
   </joint>
   <joint name="gripper_prismatic_joint_2" type="prismatic">
-    <origin rpy="0 0 3.1415" xyz="0 0 0"/>
+    <origin rpy="0 0 0" xyz="0 0 0"/>
     <parent link="gripper_rail_link"/>
     <child link="gripper_2_link"/>
     <mimic joint="gripper_prismatic_joint_1"/>
-    <axis xyz="0 -1 0"/>
+    <axis xyz="0 1 0"/>
     <limit effort="0" lower="0" upper="0.027" velocity="0.5"/>
   </joint>
@@ -1180,14 +1213,4 @@
     </actuator>
   </transmission>
-  <transmission name="tran6">
-    <type>transmission_interface/SimpleTransmission</type>
-    <joint name="joint_6">
-      <hardwareInterface>hardware_interface/EffortJointInterface</hardwareInterface>
-    </joint>
-    <actuator name="motor6">
-      <hardwareInterface>hardware_interface/EffortJointInterface</hardwareInterface>
-      <mechanicalReduction>1</mechanicalReduction>
-    </actuator>
-  </transmission>
   <transmission name="tran7">
     <type>transmission_interface/SimpleTransmission</type>
@@ -1238,5 +1261,5 @@
     <sensor name="sick_lms_5_laser_gazebo_v0" type="ray">
       <always_on>true</always_on>
-      <update_rate>50.0</update_rate>
+      <update_rate>15.0</update_rate>
       <pose>0 0 0 0 0 0</pose>
       <visualize>false</visualize>
@@ -1246,5 +1269,5 @@
             <samples>811</samples>
             <resolution>1</resolution>
-            <min_angle>-1.5708</min_angle>
+            <min_angle>-1.0</min_angle>
             <!--90 moires -->
             <max_angle>2.357</max_angle>
@@ -1253,5 +1276,5 @@
         </scan>
         <range>
-          <min>0.05</min>
+          <min>0.15</min>
           <max>4.0</max>
           <resolution>0.01</resolution>
@@ -1261,5 +1284,5 @@
         <gaussianNoise>0.005</gaussianNoise>
         <alwaysOn>true</alwaysOn>
-        <updateRate>50.0</updateRate>
+        <updateRate>15.0</updateRate>
         <topicName>scan_L</topicName>
         <frameName>sick_L_laser</frameName>
@@ -1271,5 +1294,5 @@
     <sensor name="sick_lms_5_laser_gazebo_v01" type="ray">
       <always_on>true</always_on>
-      <update_rate>50.0</update_rate>
+      <update_rate>15.0</update_rate>
       <pose>0 0 0 0 0 0</pose>
       <visualize>false</visualize>
@@ -1281,10 +1304,10 @@
             <min_angle>-2.357</min_angle>
             <!--140 moires -->
-            <max_angle>1.5708</max_angle>
+            <max_angle>1.0</max_angle>
             <!--90 moires -->
           </horizontal>
         </scan>
         <range>
-          <min>0.05</min>
+          <min>0.15</min>
           <max>4.0</max>
           <resolution>0.01</resolution>
@@ -1294,7 +1317,6 @@
         <gaussianNoise>0.005</gaussianNoise>
         <alwaysOn>true</alwaysOn>
-        <updateRate>50.0</updateRate>
+        <updateRate>15.0</updateRate>
         <topicName>scan_R</topicName>
-        <!-- allakse ta topics nomizw pws prepei na mpoun ws scan kai ta duo(scan_L & scan_R) -->
         <frameName>sick_R_laser</frameName>
       </plugin>
