Commit message: increased stability 1.0

File: demo_navi/src/urdf/model.urdf.xacro (robot description, xacro)
@@ -255,5 +255,5 @@
       <origin xyz="0 0 0"/>
       <mass value="1"/>
-      <inertia ixx="0.0007" ixy="0" ixz="0" iyy="0.0007" iyz="0" izz="0.0008"/>
+      <inertia ixx="0.000007" ixy="0" ixz="0" iyy="0.000007" iyz="0" izz="0.000008"/>
     </inertial>
     <visual>
@@ -282,5 +282,5 @@
     <inertial>
       <mass value="0.1"/>
-      <inertia ixx="6.8e-05" ixy="0" ixz="0" iyy="6.8e-05" iyz="0" izz="0.000101"/>
+      <inertia ixx="6.008e-05" ixy="0" ixz="0" iyy="6.008e-05" iyz="0" izz="0.00000101"/>
     </inertial>
     <visual>
@@ -305,10 +305,10 @@
   </joint>
   <gazebo reference="roller_s_rim_left_link">
-    <!--<mu1>5000.0</mu1>
-  				<mu2>2500.0</mu2>
-      			<kp  value="10000000.0" />
-      			<maxContacts  value="10" />
-      			<kd  value="1.0" />
-      			<fdir1 value="1 0 0"/>-->
+    <mu1>50.0</mu1>
+    <mu2>25.0</mu2>
+    <!--<kp  value="10000000.0" />
+      		<kd  value="10000000.0" />
+    	  	<dampingFactor>10</dampingFactor>
+    		<minDepth>0.001</minDepth>-->
     <material>Gazebo/Grey</material>
   </gazebo>
@@ -320,5 +320,5 @@
     <inertial>
       <mass value="0.1"/>
-      <inertia ixx="6.8e-05" ixy="0" ixz="0" iyy="6.8e-05" iyz="0" izz="0.000101"/>
+      <inertia ixx="6.008e-05" ixy="0" ixz="0" iyy="6.008e-05" iyz="0" izz="0.00000101"/>
     </inertial>
     <visual>
@@ -343,10 +343,10 @@
   </joint>
   <gazebo reference="roller_nw_rim_left_link">
-    <!--<mu1>5000.0</mu1>
-  				<mu2>2500.0</mu2>
-      			<kp  value="10000000.0" />
-      			<maxContacts  value="10" />
-      			<kd  value="1.0" />
-      			<fdir1 value="1 0 0"/>-->
+    <mu1>50.0</mu1>
+    <mu2>25.0</mu2>
+    <!--<kp  value="10000000.0" />
+      		<kd  value="10000000.0" />
+    	  	<dampingFactor>10</dampingFactor>
+    		<minDepth>0.001</minDepth>-->
     <material>Gazebo/Grey</material>
   </gazebo>
@@ -358,5 +358,5 @@
     <inertial>
       <mass value="0.1"/>
-      <inertia ixx="6.8e-05" ixy="0" ixz="0" iyy="6.8e-05" iyz="0" izz="0.000101"/>
+      <inertia ixx="6.008e-05" ixy="0" ixz="0" iyy="6.008e-05" iyz="0" izz="0.00000101"/>
     </inertial>
     <visual>
@@ -381,10 +381,10 @@
   </joint>
   <gazebo reference="roller_ne_rim_left_link">
-    <!--<mu1>5000.0</mu1>
-  				<mu2>2500.0</mu2>
-      			<kp  value="10000000.0" />
-      			<maxContacts  value="10" />
-      			<kd  value="1.0" />
-      			<fdir1 value="1 0 0"/>-->
+    <mu1>50.0</mu1>
+    <mu2>25.0</mu2>
+    <!--<kp  value="10000000.0" />
+      		<kd  value="10000000.0" />
+    	  	<dampingFactor>10</dampingFactor>
+    		<minDepth>0.001</minDepth>-->
     <material>Gazebo/Grey</material>
   </gazebo>
@@ -396,5 +396,5 @@
     <inertial>
       <mass value="0.1"/>
-      <inertia ixx="6.8e-05" ixy="0" ixz="0" iyy="6.8e-05" iyz="0" izz="0.000101"/>
+      <inertia ixx="6.008e-05" ixy="0" ixz="0" iyy="6.008e-05" iyz="0" izz="0.00000101"/>
     </inertial>
     <visual>
@@ -419,10 +419,10 @@
   </joint>
   <gazebo reference="roller_sw_rim_left_link">
-    <!--<mu1>5000.0</mu1>
-  				<mu2>2500.0</mu2>
-      			<kp  value="10000000.0" />
-      			<maxContacts  value="10" />
-      			<kd  value="1.0" />
-      			<fdir1 value="1 0 0"/>-->
+    <mu1>50.0</mu1>
+    <mu2>25.0</mu2>
+    <!--<kp  value="10000000.0" />
+      		<kd  value="10000000.0" />
+    	  	<dampingFactor>10</dampingFactor>
+    		<minDepth>0.001</minDepth>-->
     <material>Gazebo/Grey</material>
   </gazebo>
@@ -434,5 +434,5 @@
     <inertial>
       <mass value="0.1"/>
-      <inertia ixx="6.8e-05" ixy="0" ixz="0" iyy="6.8e-05" iyz="0" izz="0.000101"/>
+      <inertia ixx="6.008e-05" ixy="0" ixz="0" iyy="6.008e-05" iyz="0" izz="0.00000101"/>
     </inertial>
     <visual>
@@ -457,10 +457,10 @@
   </joint>
   <gazebo reference="roller_n_rim_left_link">
-    <!--<mu1>5000.0</mu1>
-  				<mu2>2500.0</mu2>
-      			<kp  value="10000000.0" />
-      			<maxContacts  value="10" />
-      			<kd  value="1.0" />
-      			<fdir1 value="1 0 0"/>-->
+    <mu1>50.0</mu1>
+    <mu2>25.0</mu2>
+    <!--<kp  value="10000000.0" />
+      		<kd  value="10000000.0" />
+    	  	<dampingFactor>10</dampingFactor>
+    		<minDepth>0.001</minDepth>-->
     <material>Gazebo/Grey</material>
   </gazebo>
@@ -472,5 +472,5 @@
     <inertial>
       <mass value="0.1"/>
-      <inertia ixx="6.8e-05" ixy="0" ixz="0" iyy="6.8e-05" iyz="0" izz="0.000101"/>
+      <inertia ixx="6.008e-05" ixy="0" ixz="0" iyy="6.008e-05" iyz="0" izz="0.00000101"/>
     </inertial>
     <visual>
@@ -495,10 +495,10 @@
   </joint>
   <gazebo reference="roller_se_rim_left_link">
-    <!--<mu1>5000.0</mu1>
-  				<mu2>2500.0</mu2>
-      			<kp  value="10000000.0" />
-      			<maxContacts  value="10" />
-      			<kd  value="1.0" />
-      			<fdir1 value="1 0 0"/>-->
+    <mu1>50.0</mu1>
+    <mu2>25.0</mu2>
+    <!--<kp  value="10000000.0" />
+      		<kd  value="10000000.0" />
+    	  	<dampingFactor>10</dampingFactor>
+    		<minDepth>0.001</minDepth>-->
     <material>Gazebo/Grey</material>
   </gazebo>
@@ -517,21 +517,17 @@
     </actuator>
   </transmission>
-  <!--<gazebo reference = "rim_${name}_link">
-  				<mu1>5000.0</mu1>
-  				<mu2>2500.0</mu2>
-      			<kp  value="10000000.0" />
-      			<maxContacts  value="10" />
-      			<kd  value="1.0" />
-      			<fdir1 value="1 0 0"/>
-		</gazebo>-->
-  <!--<gazebo reference = "rim_${name}_joint">
-			<dampingFactor>10</dampingFactor>
-			<minDepth>0.001</minDepth>
-		</gazebo>-->
+  <gazebo reference="rim_left_link">
+    <mu1>50.0</mu1>
+    <mu2>25.0</mu2>
+    <!--<kp  value="10000000.0" />
+      			<kd  value="10000000.0" />
+      			<dampingFactor>10</dampingFactor>
+				<minDepth>0.001</minDepth>-->
+  </gazebo>
   <link name="rim_back_link">
     <inertial>
       <origin xyz="0 0 0"/>
       <mass value="1"/>
-      <inertia ixx="0.0007" ixy="0" ixz="0" iyy="0.0007" iyz="0" izz="0.0008"/>
+      <inertia ixx="0.000007" ixy="0" ixz="0" iyy="0.000007" iyz="0" izz="0.000008"/>
     </inertial>
     <visual>
@@ -560,5 +556,5 @@
     <inertial>
       <mass value="0.1"/>
-      <inertia ixx="6.8e-05" ixy="0" ixz="0" iyy="6.8e-05" iyz="0" izz="0.000101"/>
+      <inertia ixx="6.008e-05" ixy="0" ixz="0" iyy="6.008e-05" iyz="0" izz="0.00000101"/>
     </inertial>
     <visual>
@@ -583,10 +579,10 @@
   </joint>
   <gazebo reference="roller_s_rim_back_link">
-    <!--<mu1>5000.0</mu1>
-  				<mu2>2500.0</mu2>
-      			<kp  value="10000000.0" />
-      			<maxContacts  value="10" />
-      			<kd  value="1.0" />
-      			<fdir1 value="1 0 0"/>-->
+    <mu1>50.0</mu1>
+    <mu2>25.0</mu2>
+    <!--<kp  value="10000000.0" />
+      		<kd  value="10000000.0" />
+    	  	<dampingFactor>10</dampingFactor>
+    		<minDepth>0.001</minDepth>-->
     <material>Gazebo/Grey</material>
   </gazebo>
@@ -598,5 +594,5 @@
     <inertial>
       <mass value="0.1"/>
-      <inertia ixx="6.8e-05" ixy="0" ixz="0" iyy="6.8e-05" iyz="0" izz="0.000101"/>
+      <inertia ixx="6.008e-05" ixy="0" ixz="0" iyy="6.008e-05" iyz="0" izz="0.00000101"/>
     </inertial>
     <visual>
@@ -621,10 +617,10 @@
   </joint>
   <gazebo reference="roller_nw_rim_back_link">
-    <!--<mu1>5000.0</mu1>
-  				<mu2>2500.0</mu2>
-      			<kp  value="10000000.0" />
-      			<maxContacts  value="10" />
-      			<kd  value="1.0" />
-      			<fdir1 value="1 0 0"/>-->
+    <mu1>50.0</mu1>
+    <mu2>25.0</mu2>
+    <!--<kp  value="10000000.0" />
+      		<kd  value="10000000.0" />
+    	  	<dampingFactor>10</dampingFactor>
+    		<minDepth>0.001</minDepth>-->
     <material>Gazebo/Grey</material>
   </gazebo>
@@ -636,5 +632,5 @@
     <inertial>
       <mass value="0.1"/>
-      <inertia ixx="6.8e-05" ixy="0" ixz="0" iyy="6.8e-05" iyz="0" izz="0.000101"/>
+      <inertia ixx="6.008e-05" ixy="0" ixz="0" iyy="6.008e-05" iyz="0" izz="0.00000101"/>
     </inertial>
     <visual>
@@ -659,10 +655,10 @@
   </joint>
   <gazebo reference="roller_ne_rim_back_link">
-    <!--<mu1>5000.0</mu1>
-  				<mu2>2500.0</mu2>
-      			<kp  value="10000000.0" />
-      			<maxContacts  value="10" />
-      			<kd  value="1.0" />
-      			<fdir1 value="1 0 0"/>-->
+    <mu1>50.0</mu1>
+    <mu2>25.0</mu2>
+    <!--<kp  value="10000000.0" />
+      		<kd  value="10000000.0" />
+    	  	<dampingFactor>10</dampingFactor>
+    		<minDepth>0.001</minDepth>-->
     <material>Gazebo/Grey</material>
   </gazebo>
@@ -674,5 +670,5 @@
     <inertial>
       <mass value="0.1"/>
-      <inertia ixx="6.8e-05" ixy="0" ixz="0" iyy="6.8e-05" iyz="0" izz="0.000101"/>
+      <inertia ixx="6.008e-05" ixy="0" ixz="0" iyy="6.008e-05" iyz="0" izz="0.00000101"/>
     </inertial>
     <visual>
@@ -697,10 +693,10 @@
   </joint>
   <gazebo reference="roller_sw_rim_back_link">
-    <!--<mu1>5000.0</mu1>
-  				<mu2>2500.0</mu2>
-      			<kp  value="10000000.0" />
-      			<maxContacts  value="10" />
-      			<kd  value="1.0" />
-      			<fdir1 value="1 0 0"/>-->
+    <mu1>50.0</mu1>
+    <mu2>25.0</mu2>
+    <!--<kp  value="10000000.0" />
+      		<kd  value="10000000.0" />
+    	  	<dampingFactor>10</dampingFactor>
+    		<minDepth>0.001</minDepth>-->
     <material>Gazebo/Grey</material>
   </gazebo>
@@ -712,5 +708,5 @@
     <inertial>
       <mass value="0.1"/>
-      <inertia ixx="6.8e-05" ixy="0" ixz="0" iyy="6.8e-05" iyz="0" izz="0.000101"/>
+      <inertia ixx="6.008e-05" ixy="0" ixz="0" iyy="6.008e-05" iyz="0" izz="0.00000101"/>
     </inertial>
     <visual>
@@ -735,10 +731,10 @@
   </joint>
   <gazebo reference="roller_n_rim_back_link">
-    <!--<mu1>5000.0</mu1>
-  				<mu2>2500.0</mu2>
-      			<kp  value="10000000.0" />
-      			<maxContacts  value="10" />
-      			<kd  value="1.0" />
-      			<fdir1 value="1 0 0"/>-->
+    <mu1>50.0</mu1>
+    <mu2>25.0</mu2>
+    <!--<kp  value="10000000.0" />
+      		<kd  value="10000000.0" />
+    	  	<dampingFactor>10</dampingFactor>
+    		<minDepth>0.001</minDepth>-->
     <material>Gazebo/Grey</material>
   </gazebo>
@@ -750,5 +746,5 @@
     <inertial>
       <mass value="0.1"/>
-      <inertia ixx="6.8e-05" ixy="0" ixz="0" iyy="6.8e-05" iyz="0" izz="0.000101"/>
+      <inertia ixx="6.008e-05" ixy="0" ixz="0" iyy="6.008e-05" iyz="0" izz="0.00000101"/>
     </inertial>
     <visual>
@@ -773,10 +769,10 @@
   </joint>
   <gazebo reference="roller_se_rim_back_link">
-    <!--<mu1>5000.0</mu1>
-  				<mu2>2500.0</mu2>
-      			<kp  value="10000000.0" />
-      			<maxContacts  value="10" />
-      			<kd  value="1.0" />
-      			<fdir1 value="1 0 0"/>-->
+    <mu1>50.0</mu1>
+    <mu2>25.0</mu2>
+    <!--<kp  value="10000000.0" />
+      		<kd  value="10000000.0" />
+    	  	<dampingFactor>10</dampingFactor>
+    		<minDepth>0.001</minDepth>-->
     <material>Gazebo/Grey</material>
   </gazebo>
@@ -795,21 +791,17 @@
     </actuator>
   </transmission>
-  <!--<gazebo reference = "rim_${name}_link">
-  				<mu1>5000.0</mu1>
-  				<mu2>2500.0</mu2>
-      			<kp  value="10000000.0" />
-      			<maxContacts  value="10" />
-      			<kd  value="1.0" />
-      			<fdir1 value="1 0 0"/>
-		</gazebo>-->
-  <!--<gazebo reference = "rim_${name}_joint">
-			<dampingFactor>10</dampingFactor>
-			<minDepth>0.001</minDepth>
-		</gazebo>-->
+  <gazebo reference="rim_back_link">
+    <mu1>50.0</mu1>
+    <mu2>25.0</mu2>
+    <!--<kp  value="10000000.0" />
+      			<kd  value="10000000.0" />
+      			<dampingFactor>10</dampingFactor>
+				<minDepth>0.001</minDepth>-->
+  </gazebo>
   <link name="rim_right_link">
     <inertial>
       <origin xyz="0 0 0"/>
       <mass value="1"/>
-      <inertia ixx="0.0007" ixy="0" ixz="0" iyy="0.0007" iyz="0" izz="0.0008"/>
+      <inertia ixx="0.000007" ixy="0" ixz="0" iyy="0.000007" iyz="0" izz="0.000008"/>
     </inertial>
     <visual>
@@ -838,5 +830,5 @@
     <inertial>
       <mass value="0.1"/>
-      <inertia ixx="6.8e-05" ixy="0" ixz="0" iyy="6.8e-05" iyz="0" izz="0.000101"/>
+      <inertia ixx="6.008e-05" ixy="0" ixz="0" iyy="6.008e-05" iyz="0" izz="0.00000101"/>
     </inertial>
     <visual>
@@ -861,10 +853,10 @@
   </joint>
   <gazebo reference="roller_s_rim_right_link">
-    <!--<mu1>5000.0</mu1>
-  				<mu2>2500.0</mu2>
-      			<kp  value="10000000.0" />
-      			<maxContacts  value="10" />
-      			<kd  value="1.0" />
-      			<fdir1 value="1 0 0"/>-->
+    <mu1>50.0</mu1>
+    <mu2>25.0</mu2>
+    <!--<kp  value="10000000.0" />
+      		<kd  value="10000000.0" />
+    	  	<dampingFactor>10</dampingFactor>
+    		<minDepth>0.001</minDepth>-->
     <material>Gazebo/Grey</material>
   </gazebo>
@@ -876,5 +868,5 @@
     <inertial>
       <mass value="0.1"/>
-      <inertia ixx="6.8e-05" ixy="0" ixz="0" iyy="6.8e-05" iyz="0" izz="0.000101"/>
+      <inertia ixx="6.008e-05" ixy="0" ixz="0" iyy="6.008e-05" iyz="0" izz="0.00000101"/>
     </inertial>
     <visual>
@@ -899,10 +891,10 @@
   </joint>
   <gazebo reference="roller_nw_rim_right_link">
-    <!--<mu1>5000.0</mu1>
-  				<mu2>2500.0</mu2>
-      			<kp  value="10000000.0" />
-      			<maxContacts  value="10" />
-      			<kd  value="1.0" />
-      			<fdir1 value="1 0 0"/>-->
+    <mu1>50.0</mu1>
+    <mu2>25.0</mu2>
+    <!--<kp  value="10000000.0" />
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
File: demo_navi/src/urdf/xacro/main.urdf.xacro (robot description, xacro)
@@ -140,6 +140,6 @@
          <inertial>
           <origin xyz="0 0 0" rpy="0 0 0" />
-            <mass value="0.01" />
-            <inertia ixx="0.01" ixy="0.0" ixz="0.0" iyy="0.01" iyz="0.0" izz="0.01" />
+            <mass value="0.001" />
+            <inertia ixx="0.001" ixy="0.0" ixz="0.0" iyy="0.001" iyz="0.0" izz="0.001" />
          </inertial>
       </link>
@@ -160,6 +160,6 @@
          <inertial>
           <origin xyz="0.04825 0 0.14" rpy="0 0 0" />
-            <mass value="0.01" />
-            <inertia ixx="0.01" ixy="0.0" ixz="0.0" iyy="0.01" iyz="0.0" izz="0.01" />
+            <mass value="0.001" />
+            <inertia ixx="0.001" ixy="0.0" ixz="0.0" iyy="0.001" iyz="0.0" izz="0.001" />
          </inertial>
       </link>
@@ -180,6 +180,6 @@
          <inertial>
           <origin xyz="0 0 0.14203" rpy="0 0 0" />
-            <mass value="0.01" />
-            <inertia ixx="0.01" ixy="0.0" ixz="0.0" iyy="0.01" iyz="0.0" izz="0.01"/>
+            <mass value="0.001" />
+            <inertia ixx="0.001" ixy="0.0" ixz="0.0" iyy="0.001" iyz="0.0" izz="0.001"/>
          </inertial>
       </link>
@@ -200,6 +200,6 @@
          <inertial>
           <origin xyz="0 0 0" rpy="0 0 0" />
-            <mass value="0.01" />
-            <inertia ixx="0.01" ixy="0.0" ixz="0.0" iyy="0.01" iyz="0.0" izz="0.01" />
+            <mass value="0.001" />
+            <inertia ixx="0.001" ixy="0.0" ixz="0.0" iyy="0.001" iyz="0.0" izz="0.001" />
          </inertial>
       </link>
@@ -220,6 +220,6 @@
          <inertial>
           <origin xyz="0 0 0.043" rpy="0 0 0" />
-            <mass value="0.01" />
-            <inertia ixx="0.01" ixy="0.0" ixz="0.0" iyy="0.01" iyz="0.0" izz="0.01" />
+            <mass value="0.001" />
+            <inertia ixx="0.001" ixy="0.0" ixz="0.0" iyy="0.001" iyz="0.0" izz="0.001" />
          </inertial>
       </link>
@@ -240,6 +240,6 @@
          <inertial>
           <origin xyz = "0 0 0" rpy="0 0 1.57" />
-            <mass value="0.01" />
-            <inertia ixx="0.01" ixy="0.0" ixz="0.0" iyy="0.01" iyz="0.0" izz="0.01" />
+            <mass value="0.001" />
+            <inertia ixx="0.001" ixy="0.0" ixz="0.0" iyy="0.001" iyz="0.0" izz="0.001" />
          </inertial>
       </link>
@@ -262,6 +262,6 @@
          <inertial>
           <origin xyz="0 -0.0007 0" rpy="0 0 1.57" />
-            <mass value="0.01" />
-            <inertia ixx="0.01" ixy="0.0" ixz="0.0" iyy="0.01" iyz="0.0" izz="0.01" />
+            <mass value="0.001" />
+            <inertia ixx="0.001" ixy="0.0" ixz="0.0" iyy="0.001" iyz="0.0" izz="0.001" />
          </inertial>
       </link>
@@ -282,6 +282,6 @@
          <inertial>
           <origin xyz="0 0.0007 0" rpy="0 0 -1.57" />
-            <mass value="0.01" />
-            <inertia ixx="0.01" ixy="0.0" ixz="0.0" iyy="0.01" iyz="0.0" izz="0.01" />
+            <mass value="0.001" />
+            <inertia ixx="0.001" ixy="0.0" ixz="0.0" iyy="0.001" iyz="0.0" izz="0.001" />
          </inertial>
       </link>

File: demo_navi/src/urdf/xacro/rim.urdf.xacro (robot description, xacro)
@@ -12,10 +12,10 @@
 				<mass value="1"/>
 				<inertia
-					ixx="0.0007"
+					ixx="0.000007"
 					ixy="0"
 					ixz="0"
-					iyy="0.0007"
+					iyy="0.000007"
 					iyz="0"
-					izz="0.0008"
+					izz="0.000008"
 				/>
 			</inertial>
@@ -94,16 +94,12 @@
 			</actuator>
 		</transmission>
-		<!--<gazebo reference = "rim_${name}_link">
-  				<mu1>5000.0</mu1>
-  				<mu2>2500.0</mu2>
-      			<kp  value="10000000.0" />
-      			<maxContacts  value="10" />
-      			<kd  value="1.0" />
-      			<fdir1 value="1 0 0"/>
-		</gazebo>-->
-		<!--<gazebo reference = "rim_${name}_joint">
-			<dampingFactor>10</dampingFactor>
-			<minDepth>0.001</minDepth>
-		</gazebo>-->
+		<gazebo reference = "rim_${name}_link">
+  				<mu1>50.0</mu1>
+  				<mu2>25.0</mu2>
+      			<!--<kp  value="10000000.0" />
+      			<kd  value="10000000.0" />
+      			<dampingFactor>10</dampingFactor>
+				<minDepth>0.001</minDepth>-->
+		</gazebo>
 	</xacro:macro>
 </robot>

File: demo_navi/src/urdf/xacro/roller.urdf.xacro (robot description, xacro)
@@ -9,10 +9,10 @@
 				<mass value="0.1"/>
 				<inertia
-					ixx="6.8e-05"
+					ixx="6.008e-05"
 					ixy="0"
 					ixz="0"
-					iyy="6.8e-05"
+					iyy="6.008e-05"
 					iyz="0"
-					izz="0.000101"
+					izz="0.00000101"
 				/>
 			</inertial>
@@ -44,10 +44,10 @@
 		</joint>
 	<gazebo reference="roller_${name}_rim_${parent}_link">
-  				<!--<mu1>5000.0</mu1>
-  				<mu2>2500.0</mu2>
-      			<kp  value="10000000.0" />
-      			<maxContacts  value="10" />
-      			<kd  value="1.0" />
-      			<fdir1 value="1 0 0"/>-->
+  			<mu1>50.0</mu1>
+  			<mu2>25.0</mu2>
+      		<!--<kp  value="10000000.0" />
+      		<kd  value="10000000.0" />
+    	  	<dampingFactor>10</dampingFactor>
+    		<minDepth>0.001</minDepth>-->
     <material>Gazebo/Grey</material>
   </gazebo>
