Commit message: fixed camera pos

File: demo_navi/src/urdf/model.urdf.xacro (robot description, xacro)
@@ -10,5 +10,5 @@
   <!-- camera body, with origin at bottom screw mount -->
   <joint name="camera_joint" type="fixed">
-    <origin rpy="0 -1.5708 0" xyz="-0.04 0 0.02"/>
+    <origin rpy="0 0 0" xyz="0.02 0 0.01"/>
     <parent link="wrist_2_link"/>
     <child link="camera_bottom_screw_frame"/>
@@ -224,7 +224,8 @@
   </gazebo>
   <link name="base_footprint"/>
+  <link name="imu_link"/>
   <link name="base_link">
     <inertial>
-      <origin rpy="0 0 0" xyz="-0.147 0 0"/>
+      <origin rpy="0 0 0" xyz="-0.147 0 0.05"/>
       <mass value="5"/>
       <inertia ixx="0.15" ixy="0" ixz="0" iyy="0.104167" iyz="0" izz="0.254167"/>
@@ -251,4 +252,9 @@
     <origin xyz="0 0 0"/>
   </joint>
+  <joint name="imu_joint" type="fixed">
+    <parent link="base_footprint"/>
+    <child link="imu_link"/>
+    <origin xyz="-0.145 0 0.091"/>
+  </joint>
   <link name="rim_left_link">
     <inertial>
@@ -262,5 +268,5 @@
       </geometry>
       <material name="rim_left_material">
-        <color rgba="0.3 0 0 1"/>
+        <color rgba="1.3 0 0 1"/>
       </material>
     </visual>
@@ -276,11 +282,11 @@
     <axis xyz="1 0 0"/>
     <origin rpy="0 0 -2.0944" xyz="-0.0267 0.214 0.04"/>
-    <!--<limit effort="100000" velocity="100000"/>
-			<joint_properties friction="1.0"/>-->
+    <limit effort="100000" velocity="100000"/>
+    <joint_properties friction="1.0"/>
   </joint>
   <link name="roller_s_rim_left_link">
     <inertial>
       <mass value="0.1"/>
-      <inertia ixx="6.008e-05" ixy="0" ixz="0" iyy="6.008e-05" iyz="0" izz="0.00000101"/>
+      <inertia ixx="6.008e-07" ixy="0" ixz="0" iyy="6.008e-07" iyz="0" izz="0.0000000101"/>
     </inertial>
     <visual>
@@ -303,14 +309,17 @@
     <axis xyz="0 1 0"/>
     <origin rpy="0 0 0" xyz="0.0153 0 -0.0266"/>
+    <limit effort="100000000" velocity="1000000000"/>
+    <joint_properties friction="1.0"/>
   </joint>
   <gazebo reference="roller_s_rim_left_link">
     <mu1>50.0</mu1>
     <mu2>25.0</mu2>
-    <!--<kp  value="10000000.0" />
-      		<kd  value="10000000.0" />
-    	  	<dampingFactor>10</dampingFactor>
-    		<minDepth>0.001</minDepth>-->
-    <material>Gazebo/Grey</material>
-  </gazebo>
+    <kp value="10000000000.0"/>
+    <kd value="10000000000.0"/>
+    <dampingFactor>10</dampingFactor>
+    <minDepth>0.001</minDepth>
+    <material>Gazebo/Grey</material>
+  </gazebo>
+  <selfCollide>False</selfCollide>
   <!--<gazebo reference="roller_${name}_rim_${parent}_joint">
     <dampingFactor>10</dampingFactor>
@@ -320,5 +329,5 @@
     <inertial>
       <mass value="0.1"/>
-      <inertia ixx="6.008e-05" ixy="0" ixz="0" iyy="6.008e-05" iyz="0" izz="0.00000101"/>
+      <inertia ixx="6.008e-07" ixy="0" ixz="0" iyy="6.008e-07" iyz="0" izz="0.0000000101"/>
     </inertial>
     <visual>
@@ -341,14 +350,17 @@
     <axis xyz="0 1 0"/>
     <origin rpy="1.0472 0 0" xyz="0.015 -0.0231 0.0131"/>
+    <limit effort="100000000" velocity="1000000000"/>
+    <joint_properties friction="1.0"/>
   </joint>
   <gazebo reference="roller_nw_rim_left_link">
     <mu1>50.0</mu1>
     <mu2>25.0</mu2>
-    <!--<kp  value="10000000.0" />
-      		<kd  value="10000000.0" />
-    	  	<dampingFactor>10</dampingFactor>
-    		<minDepth>0.001</minDepth>-->
-    <material>Gazebo/Grey</material>
-  </gazebo>
+    <kp value="10000000000.0"/>
+    <kd value="10000000000.0"/>
+    <dampingFactor>10</dampingFactor>
+    <minDepth>0.001</minDepth>
+    <material>Gazebo/Grey</material>
+  </gazebo>
+  <selfCollide>False</selfCollide>
   <!--<gazebo reference="roller_${name}_rim_${parent}_joint">
     <dampingFactor>10</dampingFactor>
@@ -358,5 +370,5 @@
     <inertial>
       <mass value="0.1"/>
-      <inertia ixx="6.008e-05" ixy="0" ixz="0" iyy="6.008e-05" iyz="0" izz="0.00000101"/>
+      <inertia ixx="6.008e-07" ixy="0" ixz="0" iyy="6.008e-07" iyz="0" izz="0.0000000101"/>
     </inertial>
     <visual>
@@ -379,14 +391,17 @@
     <axis xyz="0 1 0"/>
     <origin rpy="-1.0472 0 0" xyz="0.015 0.0231 0.0135"/>
+    <limit effort="100000000" velocity="1000000000"/>
+    <joint_properties friction="1.0"/>
   </joint>
   <gazebo reference="roller_ne_rim_left_link">
     <mu1>50.0</mu1>
     <mu2>25.0</mu2>
-    <!--<kp  value="10000000.0" />
-      		<kd  value="10000000.0" />
-    	  	<dampingFactor>10</dampingFactor>
-    		<minDepth>0.001</minDepth>-->
-    <material>Gazebo/Grey</material>
-  </gazebo>
+    <kp value="10000000000.0"/>
+    <kd value="10000000000.0"/>
+    <dampingFactor>10</dampingFactor>
+    <minDepth>0.001</minDepth>
+    <material>Gazebo/Grey</material>
+  </gazebo>
+  <selfCollide>False</selfCollide>
   <!--<gazebo reference="roller_${name}_rim_${parent}_joint">
     <dampingFactor>10</dampingFactor>
@@ -396,5 +411,5 @@
     <inertial>
       <mass value="0.1"/>
-      <inertia ixx="6.008e-05" ixy="0" ixz="0" iyy="6.008e-05" iyz="0" izz="0.00000101"/>
+      <inertia ixx="6.008e-07" ixy="0" ixz="0" iyy="6.008e-07" iyz="0" izz="0.0000000101"/>
     </inertial>
     <visual>
@@ -417,14 +432,17 @@
     <axis xyz="0 1 0"/>
     <origin rpy="1.0472 0 0" xyz="-0.0146 0.023 -0.0133"/>
+    <limit effort="100000000" velocity="1000000000"/>
+    <joint_properties friction="1.0"/>
   </joint>
   <gazebo reference="roller_sw_rim_left_link">
     <mu1>50.0</mu1>
     <mu2>25.0</mu2>
-    <!--<kp  value="10000000.0" />
-      		<kd  value="10000000.0" />
-    	  	<dampingFactor>10</dampingFactor>
-    		<minDepth>0.001</minDepth>-->
-    <material>Gazebo/Grey</material>
-  </gazebo>
+    <kp value="10000000000.0"/>
+    <kd value="10000000000.0"/>
+    <dampingFactor>10</dampingFactor>
+    <minDepth>0.001</minDepth>
+    <material>Gazebo/Grey</material>
+  </gazebo>
+  <selfCollide>False</selfCollide>
   <!--<gazebo reference="roller_${name}_rim_${parent}_joint">
     <dampingFactor>10</dampingFactor>
@@ -434,5 +452,5 @@
     <inertial>
       <mass value="0.1"/>
-      <inertia ixx="6.008e-05" ixy="0" ixz="0" iyy="6.008e-05" iyz="0" izz="0.00000101"/>
+      <inertia ixx="6.008e-07" ixy="0" ixz="0" iyy="6.008e-07" iyz="0" izz="0.0000000101"/>
     </inertial>
     <visual>
@@ -455,14 +473,17 @@
     <axis xyz="0 1 0"/>
     <origin rpy="0 0 0" xyz="-0.0146 0 0.0268"/>
+    <limit effort="100000000" velocity="1000000000"/>
+    <joint_properties friction="1.0"/>
   </joint>
   <gazebo reference="roller_n_rim_left_link">
     <mu1>50.0</mu1>
     <mu2>25.0</mu2>
-    <!--<kp  value="10000000.0" />
-      		<kd  value="10000000.0" />
-    	  	<dampingFactor>10</dampingFactor>
-    		<minDepth>0.001</minDepth>-->
-    <material>Gazebo/Grey</material>
-  </gazebo>
+    <kp value="10000000000.0"/>
+    <kd value="10000000000.0"/>
+    <dampingFactor>10</dampingFactor>
+    <minDepth>0.001</minDepth>
+    <material>Gazebo/Grey</material>
+  </gazebo>
+  <selfCollide>False</selfCollide>
   <!--<gazebo reference="roller_${name}_rim_${parent}_joint">
     <dampingFactor>10</dampingFactor>
@@ -472,5 +493,5 @@
     <inertial>
       <mass value="0.1"/>
-      <inertia ixx="6.008e-05" ixy="0" ixz="0" iyy="6.008e-05" iyz="0" izz="0.00000101"/>
+      <inertia ixx="6.008e-07" ixy="0" ixz="0" iyy="6.008e-07" iyz="0" izz="0.0000000101"/>
     </inertial>
     <visual>
@@ -493,14 +514,17 @@
     <axis xyz="0 1 0"/>
     <origin rpy="-1.0472 0 0" xyz="-0.0146 -0.023 -0.0133"/>
+    <limit effort="100000000" velocity="1000000000"/>
+    <joint_properties friction="1.0"/>
   </joint>
   <gazebo reference="roller_se_rim_left_link">
     <mu1>50.0</mu1>
     <mu2>25.0</mu2>
-    <!--<kp  value="10000000.0" />
-      		<kd  value="10000000.0" />
-    	  	<dampingFactor>10</dampingFactor>
-    		<minDepth>0.001</minDepth>-->
-    <material>Gazebo/Grey</material>
-  </gazebo>
+    <kp value="10000000000.0"/>
+    <kd value="10000000000.0"/>
+    <dampingFactor>10</dampingFactor>
+    <minDepth>0.001</minDepth>
+    <material>Gazebo/Grey</material>
+  </gazebo>
+  <selfCollide>False</selfCollide>
   <!--<gazebo reference="roller_${name}_rim_${parent}_joint">
     <dampingFactor>10</dampingFactor>
@@ -520,8 +544,9 @@
     <mu1>50.0</mu1>
     <mu2>25.0</mu2>
-    <!--<kp  value="10000000.0" />
+    <selfCollide>False</selfCollide>
+    <!--kp  value="10000000.0" />
       			<kd  value="10000000.0" />
       			<dampingFactor>10</dampingFactor>
-				<minDepth>0.001</minDepth>-->
+				<minDepth>0.001</minDepth-->
   </gazebo>
   <link name="rim_back_link">
@@ -536,5 +561,5 @@
       </geometry>
       <material name="rim_back_material">
-        <color rgba="0.3 0 0 1"/>
+        <color rgba="1.3 0 0 1"/>
       </material>
     </visual>
@@ -550,11 +575,11 @@
     <axis xyz="1 0 0"/>
     <origin rpy="0 0 0" xyz="-0.397 0 0.04"/>
-    <!--<limit effort="100000" velocity="100000"/>
-			<joint_properties friction="1.0"/>-->
+    <limit effort="100000" velocity="100000"/>
+    <joint_properties friction="1.0"/>
   </joint>
   <link name="roller_s_rim_back_link">
     <inertial>
       <mass value="0.1"/>
-      <inertia ixx="6.008e-05" ixy="0" ixz="0" iyy="6.008e-05" iyz="0" izz="0.00000101"/>
+      <inertia ixx="6.008e-07" ixy="0" ixz="0" iyy="6.008e-07" iyz="0" izz="0.0000000101"/>
     </inertial>
     <visual>
@@ -577,14 +602,17 @@
     <axis xyz="0 1 0"/>
     <origin rpy="0 0 0" xyz="0.0153 0 -0.0266"/>
+    <limit effort="100000000" velocity="1000000000"/>
+    <joint_properties friction="1.0"/>
   </joint>
   <gazebo reference="roller_s_rim_back_link">
     <mu1>50.0</mu1>
     <mu2>25.0</mu2>
-    <!--<kp  value="10000000.0" />
-      		<kd  value="10000000.0" />
-    	  	<dampingFactor>10</dampingFactor>
-    		<minDepth>0.001</minDepth>-->
-    <material>Gazebo/Grey</material>
-  </gazebo>
+    <kp value="10000000000.0"/>
+    <kd value="10000000000.0"/>
+    <dampingFactor>10</dampingFactor>
+    <minDepth>0.001</minDepth>
+    <material>Gazebo/Grey</material>
+  </gazebo>
+  <selfCollide>False</selfCollide>
   <!--<gazebo reference="roller_${name}_rim_${parent}_joint">
     <dampingFactor>10</dampingFactor>
@@ -594,5 +622,5 @@
     <inertial>
       <mass value="0.1"/>
-      <inertia ixx="6.008e-05" ixy="0" ixz="0" iyy="6.008e-05" iyz="0" izz="0.00000101"/>
+      <inertia ixx="6.008e-07" ixy="0" ixz="0" iyy="6.008e-07" iyz="0" izz="0.0000000101"/>
     </inertial>
     <visual>
@@ -615,14 +643,17 @@
     <axis xyz="0 1 0"/>
     <origin rpy="1.0472 0 0" xyz="0.015 -0.0231 0.0131"/>
+    <limit effort="100000000" velocity="1000000000"/>
+    <joint_properties friction="1.0"/>
   </joint>
   <gazebo reference="roller_nw_rim_back_link">
     <mu1>50.0</mu1>
     <mu2>25.0</mu2>
-    <!--<kp  value="10000000.0" />
-      		<kd  value="10000000.0" />
-    	  	<dampingFactor>10</dampingFactor>
-    		<minDepth>0.001</minDepth>-->
-    <material>Gazebo/Grey</material>
-  </gazebo>
+    <kp value="10000000000.0"/>
+    <kd value="10000000000.0"/>
+    <dampingFactor>10</dampingFactor>
+    <minDepth>0.001</minDepth>
+    <material>Gazebo/Grey</material>
+  </gazebo>
+  <selfCollide>False</selfCollide>
   <!--<gazebo reference="roller_${name}_rim_${parent}_joint">
     <dampingFactor>10</dampingFactor>
@@ -632,5 +663,5 @@
     <inertial>
       <mass value="0.1"/>
-      <inertia ixx="6.008e-05" ixy="0" ixz="0" iyy="6.008e-05" iyz="0" izz="0.00000101"/>
+      <inertia ixx="6.008e-07" ixy="0" ixz="0" iyy="6.008e-07" iyz="0" izz="0.0000000101"/>
     </inertial>
     <visual>
@@ -653,14 +684,17 @@
     <axis xyz="0 1 0"/>
     <origin rpy="-1.0472 0 0" xyz="0.015 0.0231 0.0135"/>
+    <limit effort="100000000" velocity="1000000000"/>
+    <joint_properties friction="1.0"/>
   </joint>
   <gazebo reference="roller_ne_rim_back_link">
     <mu1>50.0</mu1>
     <mu2>25.0</mu2>
-    <!--<kp  value="10000000.0" />
-      		<kd  value="10000000.0" />
-    	  	<dampingFactor>10</dampingFactor>
-    		<minDepth>0.001</minDepth>-->
-    <material>Gazebo/Grey</material>
-  </gazebo>
+    <kp value="10000000000.0"/>
+    <kd value="10000000000.0"/>
+    <dampingFactor>10</dampingFactor>
+    <minDepth>0.001</minDepth>
+    <material>Gazebo/Grey</material>
+  </gazebo>
+  <selfCollide>False</selfCollide>
   <!--<gazebo reference="roller_${name}_rim_${parent}_joint">
     <dampingFactor>10</dampingFactor>
@@ -670,5 +704,5 @@
     <inertial>
       <mass value="0.1"/>
-      <inertia ixx="6.008e-05" ixy="0" ixz="0" iyy="6.008e-05" iyz="0" izz="0.00000101"/>
+      <inertia ixx="6.008e-07" ixy="0" ixz="0" iyy="6.008e-07" iyz="0" izz="0.0000000101"/>
     </inertial>
     <visual>
@@ -691,14 +725,17 @@
     <axis xyz="0 1 0"/>
     <origin rpy="1.0472 0 0" xyz="-0.0146 0.023 -0.0133"/>
+    <limit effort="100000000" velocity="1000000000"/>
+    <joint_properties friction="1.0"/>
   </joint>
   <gazebo reference="roller_sw_rim_back_link">
     <mu1>50.0</mu1>
     <mu2>25.0</mu2>
-    <!--<kp  value="10000000.0" />
-      		<kd  value="10000000.0" />
-    	  	<dampingFactor>10</dampingFactor>
-    		<minDepth>0.001</minDepth>-->
-    <material>Gazebo/Grey</material>
-  </gazebo>
+    <kp value="10000000000.0"/>
+    <kd value="10000000000.0"/>
+    <dampingFactor>10</dampingFactor>
+    <minDepth>0.001</minDepth>
+    <material>Gazebo/Grey</material>
+  </gazebo>
+  <selfCollide>False</selfCollide>
   <!--<gazebo reference="roller_${name}_rim_${parent}_joint">
     <dampingFactor>10</dampingFactor>
@@ -708,5 +745,5 @@
     <inertial>
       <mass value="0.1"/>
-      <inertia ixx="6.008e-05" ixy="0" ixz="0" iyy="6.008e-05" iyz="0" izz="0.00000101"/>
+      <inertia ixx="6.008e-07" ixy="0" ixz="0" iyy="6.008e-07" iyz="0" izz="0.0000000101"/>
     </inertial>
     <visual>
@@ -729,14 +766,17 @@
     <axis xyz="0 1 0"/>
     <origin rpy="0 0 0" xyz="-0.0146 0 0.0268"/>
+    <limit effort="100000000" velocity="1000000000"/>
+    <joint_properties friction="1.0"/>
   </joint>
   <gazebo reference="roller_n_rim_back_link">
     <mu1>50.0</mu1>
     <mu2>25.0</mu2>
-    <!--<kp  value="10000000.0" />
-      		<kd  value="10000000.0" />
-    	  	<dampingFactor>10</dampingFactor>
-    		<minDepth>0.001</minDepth>-->
-    <material>Gazebo/Grey</material>
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
File: demo_navi/src/urdf/xacro/main.urdf.xacro (robot description, xacro)
@@ -8,10 +8,11 @@
   <xacro:include filename="$(find realsense2_description)/urdf/_d435.urdf.xacro" />
   <xacro:sensor_d435 name="camera" topics_ns="camera" parent="wrist_2_link" publish_pointcloud="true">
-    <origin xyz="-0.04 0 0.02" rpy="0 -1.5708 0" />
+    <origin xyz="0.02 0 0.01" rpy="0 0 0" />
   </xacro:sensor_d435>
 	<link name="base_footprint"/>
+  <link name="imu_link"/>
 	<link name="base_link">
 	<inertial>
-		<origin xyz="-0.147 0 0"
+		<origin xyz="-0.147 0 0.05"
 			rpy="0 0 0" />
 		<mass value="5"/>
@@ -53,7 +54,17 @@
 		/>
 	</joint>
+    <joint
+    name="imu_joint"
+    type="fixed"
+  >
+    <parent link="base_footprint" />
+    <child link="imu_link"/>
+    <origin
+      xyz="-0.145 0 0.091"
+    />
+  </joint>
 	<xacro:rim_macro
 		name="left"
-		color="0.3 0 0"
+		color="1.3 0 0"
 		xyz="-0.0267 0.214 0.04"
 		rpy="0 0 -2.0944"
@@ -61,5 +72,5 @@
 	<xacro:rim_macro
 		name="back"
-		color="0.3 0 0"
+		color="1.3 0 0"
 		xyz="-0.397 0 0.04"
 		rpy="0 0 0"
@@ -67,5 +78,5 @@
 	<xacro:rim_macro
 		name="right"
-		color="0.3 0 0"
+		color="1.3 0 0"
 		xyz="-0.0267 -0.214 0.04"
 		rpy="0 0 2.0944"
@@ -90,10 +101,10 @@
         </geometry>
       </collision>
-      <inertial>
+      <!--inertial>
         <mass value="0.001" />
         <origin xyz="0.008 -0.275 0.042" />
         <inertia ixx="0.000001" ixy="0.0" ixz="0.0"
           iyy="0.000001" iyz="0.0" izz="0.000001" />
-      </inertial>
+      </inertial-->
     </link>
     <joint name="sick_joint_L" type="fixed">
@@ -116,10 +127,10 @@
         </geometry>
       </collision>
-      <inertial>
+      <!--inertial>
         <mass value="0.001" />
         <origin xyz="0 0.27 0.07" />
         <inertia ixx="0.000001" ixy="0.0" ixz="0.0"
           iyy="0.000001" iyz="0.0" izz="0.000001" />
-      </inertial>
+      </inertial-->
     </link>
     <!--WIDOWXL ARM LINKS & JOINTS-->
@@ -330,5 +341,5 @@
          <limit lower="-0.31" upper="0.1" effort="100" velocity="0.5" />
       </joint>
-            <joint name="gripper_revolute_joint" type="revolute">
+      <joint name="gripper_revolute_joint" type="revolute">
          <origin xyz = "0 0 0" rpy="0 0 0" />
          <parent link="gripper_rail_link" />
@@ -354,8 +365,8 @@
     <type>transmission_interface/SimpleTransmission</type>
     <joint name="joint_1">
-          <hardwareInterface>hardware_interface/PositionJointInterface</hardwareInterface>
+          <hardwareInterface>hardware_interface/EffortJointInterface</hardwareInterface>
     </joint>
     <actuator name="motor1">
-      <hardwareInterface>hardware_interface/PositionJointInterface</hardwareInterface>
+      <hardwareInterface>hardware_interface/EffortJointInterface</hardwareInterface>
       <mechanicalReduction>1</mechanicalReduction>
     </actuator>
@@ -364,8 +375,8 @@
     <type>transmission_interface/SimpleTransmission</type>
     <joint name="joint_2">
-          <hardwareInterface>hardware_interface/PositionJointInterface</hardwareInterface>
+          <hardwareInterface>hardware_interface/EffortJointInterface</hardwareInterface>
     </joint>
     <actuator name="motor2">
-      <hardwareInterface>hardware_interface/PositionJointInterface</hardwareInterface>
+      <hardwareInterface>hardware_interface/EffortJointInterface</hardwareInterface>
       <mechanicalReduction>1</mechanicalReduction>
     </actuator>
@@ -374,8 +385,8 @@
     <type>transmission_interface/SimpleTransmission</type>
     <joint name="joint_3">
-          <hardwareInterface>hardware_interface/PositionJointInterface</hardwareInterface>
+          <hardwareInterface>hardware_interface/EffortJointInterface</hardwareInterface>
     </joint>
     <actuator name="motor3">
-      <hardwareInterface>hardware_interface/PositionJointInterface</hardwareInterface>
+      <hardwareInterface>hardware_interface/EffortJointInterface</hardwareInterface>
       <mechanicalReduction>1</mechanicalReduction>
     </actuator>
@@ -384,8 +395,8 @@
     <type>transmission_interface/SimpleTransmission</type>
     <joint name="joint_4">
-          <hardwareInterface>hardware_interface/PositionJointInterface</hardwareInterface>
+          <hardwareInterface>hardware_interface/EffortJointInterface</hardwareInterface>
     </joint>
     <actuator name="motor4">
-      <hardwareInterface>hardware_interface/PositionJointInterface</hardwareInterface>
+      <hardwareInterface>hardware_interface/EffortJointInterface</hardwareInterface>
       <mechanicalReduction>1</mechanicalReduction>
     </actuator>
@@ -394,8 +405,8 @@
     <type>transmission_interface/SimpleTransmission</type>
     <joint name="joint_5">
-          <hardwareInterface>hardware_interface/PositionJointInterface</hardwareInterface>
+          <hardwareInterface>hardware_interface/EffortJointInterface</hardwareInterface>
     </joint>
     <actuator name="motor5">
-      <hardwareInterface>hardware_interface/PositionJointInterface</hardwareInterface>
+      <hardwareInterface>hardware_interface/EffortJointInterface</hardwareInterface>
       <mechanicalReduction>1</mechanicalReduction>
     </actuator>
@@ -404,8 +415,8 @@
     <type>transmission_interface/SimpleTransmission</type>
     <joint name="gripper_prismatic_joint_1">
-          <hardwareInterface>hardware_interface/PositionJointInterface</hardwareInterface>
+          <hardwareInterface>hardware_interface/EffortJointInterface</hardwareInterface>
     </joint>
     <actuator name="motor7">
-      <hardwareInterface>hardware_interface/PositionJointInterface</hardwareInterface>
+      <hardwareInterface>hardware_interface/EffortJointInterface</hardwareInterface>
       <mechanicalReduction>1</mechanicalReduction>
     </actuator>
@@ -414,8 +425,8 @@
     <type>transmission_interface/SimpleTransmission</type>
     <joint name="gripper_prismatic_joint_2">
-          <hardwareInterface>hardware_interface/PositionJointInterface</hardwareInterface>
+          <hardwareInterface>hardware_interface/EffortJointInterface</hardwareInterface>
     </joint>
     <actuator name="motor8">
-      <hardwareInterface>hardware_interface/PositionJointInterface</hardwareInterface>
+      <hardwareInterface>hardware_interface/EffortJointInterface</hardwareInterface>
       <mechanicalReduction>1</mechanicalReduction>
     </actuator>
@@ -445,4 +456,24 @@
      </plugin>
    </gazebo>
+  <gazebo reference="imu_link">
+    <gravity>true</gravity>
+    <sensor name="imu_sensor" type="imu">
+      <always_on>true</always_on>
+      <update_rate>100</update_rate>
+      <visualize>true</visualize>
+      <topic>__default_topic__</topic>
+      <plugin filename="libgazebo_ros_imu_sensor.so" name="imu_plugin">
+        <topicName>imu</topicName>
+        <bodyName>imu_link</bodyName>
+        <updateRateHZ>10.0</updateRateHZ>
+        <gaussianNoise>0.0</gaussianNoise>
+        <xyzOffset>0 0 0</xyzOffset>
+        <rpyOffset>0 0 0</rpyOffset>
+        <frameName>imu_link</frameName>
+        <initialOrientationAsReference>false</initialOrientationAsReference>
+      </plugin>
+      <pose>0 0 0 0 0 0</pose>
+    </sensor>
+  </gazebo>
     <gazebo reference="sick_L_laser">
     <material value="Gazebo/Blue" />
@@ -507,4 +538,21 @@
     </sensor>
   </gazebo>
+  <gazebo>
+   <plugin name="gazebo_grasp_fix" filename="libgazebo_grasp_fix.so">
+        <arm>
+           <arm_name>widowxl</arm_name>
+           <palm_link>wrist_2_link</palm_link>
+           <gripper_link>gripper_1_link</gripper_link>
+           <gripper_link>gripper_2_link</gripper_link>
+        </arm>
+       <forces_angle_tolerance>100</forces_angle_tolerance>
+       <update_rate>10</update_rate>
+       <grip_count_threshold>4</grip_count_threshold>
+       <max_grip_count>30</max_grip_count>
+       <release_tolerance>0.01</release_tolerance>
+       <disable_collisions_on_attach>false</disable_collisions_on_attach>
+       <contact_topic>__default_topic__</contact_topic>
+    </plugin>
+</gazebo>
 	<gazebo reference="base_link">
     		<material>Gazebo/Crimson</material>

File: demo_navi/src/urdf/xacro/rim.urdf.xacro (robot description, xacro)
@@ -45,6 +45,6 @@
 				rpy="${rpy}"
 			/>
-			<!--<limit effort="100000" velocity="100000"/>
-			<joint_properties friction="1.0"/>-->
+			<limit effort="100000" velocity="100000"/>
+			<joint_properties friction="1.0"/>
 		</joint>
 		<xacro:roller_macro
@@ -97,8 +97,9 @@
   				<mu1>50.0</mu1>
   				<mu2>25.0</mu2>
-      			<!--<kp  value="10000000.0" />
+  				<selfCollide>False</selfCollide>
+      			<!--kp  value="10000000.0" />
       			<kd  value="10000000.0" />
       			<dampingFactor>10</dampingFactor>
-				<minDepth>0.001</minDepth>-->
+				<minDepth>0.001</minDepth-->
 		</gazebo>
 	</xacro:macro>
