Commit message: fixed camera pos

File: demo_navi/src/urdf/xacro/roller.urdf.xacro (robot description, xacro)
@@ -9,10 +9,10 @@
 				<mass value="0.1"/>
 				<inertia
-					ixx="6.008e-05"
+					ixx="6.008e-07"
 					ixy="0"
 					ixz="0"
-					iyy="6.008e-05"
+					iyy="6.008e-07"
 					iyz="0"
-					izz="0.00000101"
+					izz="0.0000000101"
 				/>
 			</inertial>
@@ -42,14 +42,17 @@
 				rpy="${rpy}"
 			/>
+			<limit effort="100000000" velocity="1000000000"/>
+			<joint_properties friction="1.0"/>
 		</joint>
 	<gazebo reference="roller_${name}_rim_${parent}_link">
   			<mu1>50.0</mu1>
   			<mu2>25.0</mu2>
-      		<!--<kp  value="10000000.0" />
-      		<kd  value="10000000.0" />
+      		<kp  value="10000000000.0" />
+      		<kd  value="10000000000.0" />
     	  	<dampingFactor>10</dampingFactor>
-    		<minDepth>0.001</minDepth>-->
+    		<minDepth>0.001</minDepth>
     <material>Gazebo/Grey</material>
   </gazebo>
+  <selfCollide>False</selfCollide>
   <!--<gazebo reference="roller_${name}_rim_${parent}_joint">
     <dampingFactor>10</dampingFactor>

Commit message: Added gripper_plugin

File: demo_navi/src/urdf/model.urdf.xacro (robot description, xacro)
@@ -10,5 +10,5 @@
   <!-- camera body, with origin at bottom screw mount -->
   <joint name="camera_joint" type="fixed">
-    <origin rpy="0 0 0" xyz="0.02 0 0.01"/>
+    <origin rpy="0 0 0" xyz="0.025 0 0.01"/>
     <parent link="wrist_2_link"/>
     <child link="camera_bottom_screw_frame"/>
@@ -229,5 +229,5 @@
       <origin rpy="0 0 0" xyz="-0.147 0 0.05"/>
       <mass value="5"/>
-      <inertia ixx="0.15" ixy="0" ixz="0" iyy="0.104167" iyz="0" izz="0.254167"/>
+      <inertia ixx="0.04" ixy="0" ixz="0" iyy="0.04" iyz="0" izz="0.08"/>
     </inertial>
     <visual>
@@ -260,5 +260,5 @@
     <inertial>
       <origin xyz="0 0 0"/>
-      <mass value="1"/>
+      <mass value="2.5"/>
       <inertia ixx="0.000007" ixy="0" ixz="0" iyy="0.000007" iyz="0" izz="0.000008"/>
     </inertial>
@@ -282,10 +282,9 @@
     <axis xyz="1 0 0"/>
     <origin rpy="0 0 -2.0944" xyz="-0.0267 0.214 0.04"/>
-    <limit effort="100000" velocity="100000"/>
-    <joint_properties friction="1.0"/>
+    <limit effort="1000000000" velocity="1000"/>
   </joint>
   <link name="roller_s_rim_left_link">
     <inertial>
-      <mass value="0.1"/>
+      <mass value="1"/>
       <inertia ixx="6.008e-07" ixy="0" ixz="0" iyy="6.008e-07" iyz="0" izz="0.0000000101"/>
     </inertial>
@@ -309,18 +308,17 @@
     <axis xyz="0 1 0"/>
     <origin rpy="0 0 0" xyz="0.0153 0 -0.0266"/>
-    <limit effort="100000000" velocity="1000000000"/>
-    <joint_properties friction="1.0"/>
+    <limit effort="100000000" velocity="1000"/>
   </joint>
   <gazebo reference="roller_s_rim_left_link">
-    <mu1>50.0</mu1>
-    <mu2>25.0</mu2>
-    <kp value="10000000000.0"/>
-    <kd value="10000000000.0"/>
-    <dampingFactor>10</dampingFactor>
-    <minDepth>0.001</minDepth>
-    <material>Gazebo/Grey</material>
-  </gazebo>
-  <selfCollide>False</selfCollide>
-  <!--<gazebo reference="roller_${name}_rim_${parent}_joint">
+    <!--<mu1>50.0</mu1>
+  			<mu2>25.0</mu2>-->
+    <kp value="10000000000.0"/>
+    <kd value="10000000000.0"/>
+    <dampingFactor>10</dampingFactor>
+    <minDepth>0.001</minDepth>
+    <material>Gazebo/Grey</material>
+  </gazebo>
+  <!--<gazebo reference="roller_${name}_rim_${parent}_joint">
+    <selfCollide>False</selfCollide>
     <dampingFactor>10</dampingFactor>
     <minDepth>0.001</minDepth>
@@ -328,5 +326,5 @@
   <link name="roller_nw_rim_left_link">
     <inertial>
-      <mass value="0.1"/>
+      <mass value="1"/>
       <inertia ixx="6.008e-07" ixy="0" ixz="0" iyy="6.008e-07" iyz="0" izz="0.0000000101"/>
     </inertial>
@@ -350,18 +348,17 @@
     <axis xyz="0 1 0"/>
     <origin rpy="1.0472 0 0" xyz="0.015 -0.0231 0.0131"/>
-    <limit effort="100000000" velocity="1000000000"/>
-    <joint_properties friction="1.0"/>
+    <limit effort="100000000" velocity="1000"/>
   </joint>
   <gazebo reference="roller_nw_rim_left_link">
-    <mu1>50.0</mu1>
-    <mu2>25.0</mu2>
-    <kp value="10000000000.0"/>
-    <kd value="10000000000.0"/>
-    <dampingFactor>10</dampingFactor>
-    <minDepth>0.001</minDepth>
-    <material>Gazebo/Grey</material>
-  </gazebo>
-  <selfCollide>False</selfCollide>
-  <!--<gazebo reference="roller_${name}_rim_${parent}_joint">
+    <!--<mu1>50.0</mu1>
+  			<mu2>25.0</mu2>-->
+    <kp value="10000000000.0"/>
+    <kd value="10000000000.0"/>
+    <dampingFactor>10</dampingFactor>
+    <minDepth>0.001</minDepth>
+    <material>Gazebo/Grey</material>
+  </gazebo>
+  <!--<gazebo reference="roller_${name}_rim_${parent}_joint">
+    <selfCollide>False</selfCollide>
     <dampingFactor>10</dampingFactor>
     <minDepth>0.001</minDepth>
@@ -369,5 +366,5 @@
   <link name="roller_ne_rim_left_link">
     <inertial>
-      <mass value="0.1"/>
+      <mass value="1"/>
       <inertia ixx="6.008e-07" ixy="0" ixz="0" iyy="6.008e-07" iyz="0" izz="0.0000000101"/>
     </inertial>
@@ -391,18 +388,17 @@
     <axis xyz="0 1 0"/>
     <origin rpy="-1.0472 0 0" xyz="0.015 0.0231 0.0135"/>
-    <limit effort="100000000" velocity="1000000000"/>
-    <joint_properties friction="1.0"/>
+    <limit effort="100000000" velocity="1000"/>
   </joint>
   <gazebo reference="roller_ne_rim_left_link">
-    <mu1>50.0</mu1>
-    <mu2>25.0</mu2>
-    <kp value="10000000000.0"/>
-    <kd value="10000000000.0"/>
-    <dampingFactor>10</dampingFactor>
-    <minDepth>0.001</minDepth>
-    <material>Gazebo/Grey</material>
-  </gazebo>
-  <selfCollide>False</selfCollide>
-  <!--<gazebo reference="roller_${name}_rim_${parent}_joint">
+    <!--<mu1>50.0</mu1>
+  			<mu2>25.0</mu2>-->
+    <kp value="10000000000.0"/>
+    <kd value="10000000000.0"/>
+    <dampingFactor>10</dampingFactor>
+    <minDepth>0.001</minDepth>
+    <material>Gazebo/Grey</material>
+  </gazebo>
+  <!--<gazebo reference="roller_${name}_rim_${parent}_joint">
+    <selfCollide>False</selfCollide>
     <dampingFactor>10</dampingFactor>
     <minDepth>0.001</minDepth>
@@ -410,5 +406,5 @@
   <link name="roller_sw_rim_left_link">
     <inertial>
-      <mass value="0.1"/>
+      <mass value="1"/>
       <inertia ixx="6.008e-07" ixy="0" ixz="0" iyy="6.008e-07" iyz="0" izz="0.0000000101"/>
     </inertial>
@@ -432,18 +428,17 @@
     <axis xyz="0 1 0"/>
     <origin rpy="1.0472 0 0" xyz="-0.0146 0.023 -0.0133"/>
-    <limit effort="100000000" velocity="1000000000"/>
-    <joint_properties friction="1.0"/>
+    <limit effort="100000000" velocity="1000"/>
   </joint>
   <gazebo reference="roller_sw_rim_left_link">
-    <mu1>50.0</mu1>
-    <mu2>25.0</mu2>
-    <kp value="10000000000.0"/>
-    <kd value="10000000000.0"/>
-    <dampingFactor>10</dampingFactor>
-    <minDepth>0.001</minDepth>
-    <material>Gazebo/Grey</material>
-  </gazebo>
-  <selfCollide>False</selfCollide>
-  <!--<gazebo reference="roller_${name}_rim_${parent}_joint">
+    <!--<mu1>50.0</mu1>
+  			<mu2>25.0</mu2>-->
+    <kp value="10000000000.0"/>
+    <kd value="10000000000.0"/>
+    <dampingFactor>10</dampingFactor>
+    <minDepth>0.001</minDepth>
+    <material>Gazebo/Grey</material>
+  </gazebo>
+  <!--<gazebo reference="roller_${name}_rim_${parent}_joint">
+    <selfCollide>False</selfCollide>
     <dampingFactor>10</dampingFactor>
     <minDepth>0.001</minDepth>
@@ -451,5 +446,5 @@
   <link name="roller_n_rim_left_link">
     <inertial>
-      <mass value="0.1"/>
+      <mass value="1"/>
       <inertia ixx="6.008e-07" ixy="0" ixz="0" iyy="6.008e-07" iyz="0" izz="0.0000000101"/>
     </inertial>
@@ -473,18 +468,17 @@
     <axis xyz="0 1 0"/>
     <origin rpy="0 0 0" xyz="-0.0146 0 0.0268"/>
-    <limit effort="100000000" velocity="1000000000"/>
-    <joint_properties friction="1.0"/>
+    <limit effort="100000000" velocity="1000"/>
   </joint>
   <gazebo reference="roller_n_rim_left_link">
-    <mu1>50.0</mu1>
-    <mu2>25.0</mu2>
-    <kp value="10000000000.0"/>
-    <kd value="10000000000.0"/>
-    <dampingFactor>10</dampingFactor>
-    <minDepth>0.001</minDepth>
-    <material>Gazebo/Grey</material>
-  </gazebo>
-  <selfCollide>False</selfCollide>
-  <!--<gazebo reference="roller_${name}_rim_${parent}_joint">
+    <!--<mu1>50.0</mu1>
+  			<mu2>25.0</mu2>-->
+    <kp value="10000000000.0"/>
+    <kd value="10000000000.0"/>
+    <dampingFactor>10</dampingFactor>
+    <minDepth>0.001</minDepth>
+    <material>Gazebo/Grey</material>
+  </gazebo>
+  <!--<gazebo reference="roller_${name}_rim_${parent}_joint">
+    <selfCollide>False</selfCollide>
     <dampingFactor>10</dampingFactor>
     <minDepth>0.001</minDepth>
@@ -492,5 +486,5 @@
   <link name="roller_se_rim_left_link">
     <inertial>
-      <mass value="0.1"/>
+      <mass value="1"/>
       <inertia ixx="6.008e-07" ixy="0" ixz="0" iyy="6.008e-07" iyz="0" izz="0.0000000101"/>
     </inertial>
@@ -514,18 +508,17 @@
     <axis xyz="0 1 0"/>
     <origin rpy="-1.0472 0 0" xyz="-0.0146 -0.023 -0.0133"/>
-    <limit effort="100000000" velocity="1000000000"/>
-    <joint_properties friction="1.0"/>
+    <limit effort="100000000" velocity="1000"/>
   </joint>
   <gazebo reference="roller_se_rim_left_link">
-    <mu1>50.0</mu1>
-    <mu2>25.0</mu2>
-    <kp value="10000000000.0"/>
-    <kd value="10000000000.0"/>
-    <dampingFactor>10</dampingFactor>
-    <minDepth>0.001</minDepth>
-    <material>Gazebo/Grey</material>
-  </gazebo>
-  <selfCollide>False</selfCollide>
-  <!--<gazebo reference="roller_${name}_rim_${parent}_joint">
+    <!--<mu1>50.0</mu1>
+  			<mu2>25.0</mu2>-->
+    <kp value="10000000000.0"/>
+    <kd value="10000000000.0"/>
+    <dampingFactor>10</dampingFactor>
+    <minDepth>0.001</minDepth>
+    <material>Gazebo/Grey</material>
+  </gazebo>
+  <!--<gazebo reference="roller_${name}_rim_${parent}_joint">
+    <selfCollide>False</selfCollide>
     <dampingFactor>10</dampingFactor>
     <minDepth>0.001</minDepth>
@@ -542,8 +535,8 @@
   </transmission>
   <gazebo reference="rim_left_link">
-    <mu1>50.0</mu1>
-    <mu2>25.0</mu2>
-    <selfCollide>False</selfCollide>
+    <!--<mu1>50.0</mu1>
+  				<mu2>25.0</mu2>-->
     <!--kp  value="10000000.0" />
+      			<selfCollide>False</selfCollide>
       			<kd  value="10000000.0" />
       			<dampingFactor>10</dampingFactor>
@@ -553,5 +546,5 @@
     <inertial>
       <origin xyz="0 0 0"/>
-      <mass value="1"/>
+      <mass value="2.5"/>
       <inertia ixx="0.000007" ixy="0" ixz="0" iyy="0.000007" iyz="0" izz="0.000008"/>
     </inertial>
@@ -575,10 +568,9 @@
     <axis xyz="1 0 0"/>
     <origin rpy="0 0 0" xyz="-0.397 0 0.04"/>
-    <limit effort="100000" velocity="100000"/>
-    <joint_properties friction="1.0"/>
+    <limit effort="1000000000" velocity="1000"/>
   </joint>
   <link name="roller_s_rim_back_link">
     <inertial>
-      <mass value="0.1"/>
+      <mass value="1"/>
       <inertia ixx="6.008e-07" ixy="0" ixz="0" iyy="6.008e-07" iyz="0" izz="0.0000000101"/>
     </inertial>
@@ -602,18 +594,17 @@
     <axis xyz="0 1 0"/>
     <origin rpy="0 0 0" xyz="0.0153 0 -0.0266"/>
-    <limit effort="100000000" velocity="1000000000"/>
-    <joint_properties friction="1.0"/>
+    <limit effort="100000000" velocity="1000"/>
   </joint>
   <gazebo reference="roller_s_rim_back_link">
-    <mu1>50.0</mu1>
-    <mu2>25.0</mu2>
-    <kp value="10000000000.0"/>
-    <kd value="10000000000.0"/>
-    <dampingFactor>10</dampingFactor>
-    <minDepth>0.001</minDepth>
-    <material>Gazebo/Grey</material>
-  </gazebo>
-  <selfCollide>False</selfCollide>
-  <!--<gazebo reference="roller_${name}_rim_${parent}_joint">
+    <!--<mu1>50.0</mu1>
+  			<mu2>25.0</mu2>-->
+    <kp value="10000000000.0"/>
+    <kd value="10000000000.0"/>
+    <dampingFactor>10</dampingFactor>
+    <minDepth>0.001</minDepth>
+    <material>Gazebo/Grey</material>
+  </gazebo>
+  <!--<gazebo reference="roller_${name}_rim_${parent}_joint">
+    <selfCollide>False</selfCollide>
     <dampingFactor>10</dampingFactor>
     <minDepth>0.001</minDepth>
@@ -621,5 +612,5 @@
   <link name="roller_nw_rim_back_link">
     <inertial>
-      <mass value="0.1"/>
+      <mass value="1"/>
       <inertia ixx="6.008e-07" ixy="0" ixz="0" iyy="6.008e-07" iyz="0" izz="0.0000000101"/>
     </inertial>
@@ -643,18 +634,17 @@
     <axis xyz="0 1 0"/>
     <origin rpy="1.0472 0 0" xyz="0.015 -0.0231 0.0131"/>
-    <limit effort="100000000" velocity="1000000000"/>
-    <joint_properties friction="1.0"/>
+    <limit effort="100000000" velocity="1000"/>
   </joint>
   <gazebo reference="roller_nw_rim_back_link">
-    <mu1>50.0</mu1>
-    <mu2>25.0</mu2>
-    <kp value="10000000000.0"/>
-    <kd value="10000000000.0"/>
-    <dampingFactor>10</dampingFactor>
-    <minDepth>0.001</minDepth>
-    <material>Gazebo/Grey</material>
-  </gazebo>
-  <selfCollide>False</selfCollide>
-  <!--<gazebo reference="roller_${name}_rim_${parent}_joint">
+    <!--<mu1>50.0</mu1>
+  			<mu2>25.0</mu2>-->
+    <kp value="10000000000.0"/>
+    <kd value="10000000000.0"/>
+    <dampingFactor>10</dampingFactor>
+    <minDepth>0.001</minDepth>
+    <material>Gazebo/Grey</material>
+  </gazebo>
+  <!--<gazebo reference="roller_${name}_rim_${parent}_joint">
+    <selfCollide>False</selfCollide>
     <dampingFactor>10</dampingFactor>
     <minDepth>0.001</minDepth>
@@ -662,5 +652,5 @@
   <link name="roller_ne_rim_back_link">
     <inertial>
-      <mass value="0.1"/>
+      <mass value="1"/>
       <inertia ixx="6.008e-07" ixy="0" ixz="0" iyy="6.008e-07" iyz="0" izz="0.0000000101"/>
     </inertial>
@@ -684,18 +674,17 @@
     <axis xyz="0 1 0"/>
     <origin rpy="-1.0472 0 0" xyz="0.015 0.0231 0.0135"/>
-    <limit effort="100000000" velocity="1000000000"/>
-    <joint_properties friction="1.0"/>
+    <limit effort="100000000" velocity="1000"/>
   </joint>
   <gazebo reference="roller_ne_rim_back_link">
-    <mu1>50.0</mu1>
-    <mu2>25.0</mu2>
-    <kp value="10000000000.0"/>
-    <kd value="10000000000.0"/>
-    <dampingFactor>10</dampingFactor>
-    <minDepth>0.001</minDepth>
-    <material>Gazebo/Grey</material>
-  </gazebo>
-  <selfCollide>False</selfCollide>
-  <!--<gazebo reference="roller_${name}_rim_${parent}_joint">
+    <!--<mu1>50.0</mu1>
+  			<mu2>25.0</mu2>-->
+    <kp value="10000000000.0"/>
+    <kd value="10000000000.0"/>
+    <dampingFactor>10</dampingFactor>
+    <minDepth>0.001</minDepth>
+    <material>Gazebo/Grey</material>
+  </gazebo>
+  <!--<gazebo reference="roller_${name}_rim_${parent}_joint">
+    <selfCollide>False</selfCollide>
     <dampingFactor>10</dampingFactor>
     <minDepth>0.001</minDepth>
@@ -703,5 +692,5 @@
   <link name="roller_sw_rim_back_link">
     <inertial>
-      <mass value="0.1"/>
+      <mass value="1"/>
       <inertia ixx="6.008e-07" ixy="0" ixz="0" iyy="6.008e-07" iyz="0" izz="0.0000000101"/>
     </inertial>
@@ -725,18 +714,17 @@
     <axis xyz="0 1 0"/>
     <origin rpy="1.0472 0 0" xyz="-0.0146 0.023 -0.0133"/>
-    <limit effort="100000000" velocity="1000000000"/>
-    <joint_properties friction="1.0"/>
+    <limit effort="100000000" velocity="1000"/>
   </joint>
   <gazebo reference="roller_sw_rim_back_link">
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
File: demo_navi/src/urdf/xacro/main.urdf.xacro (robot description, xacro)
@@ -8,5 +8,5 @@
   <xacro:include filename="$(find realsense2_description)/urdf/_d435.urdf.xacro" />
   <xacro:sensor_d435 name="camera" topics_ns="camera" parent="wrist_2_link" publish_pointcloud="true">
-    <origin xyz="0.02 0 0.01" rpy="0 0 0" />
+    <origin xyz="0.025 0 0.01" rpy="0 0 0" />
   </xacro:sensor_d435>
 	<link name="base_footprint"/>
@@ -18,10 +18,10 @@
 		<mass value="5"/>
 		<inertia
-			ixx="0.15"
+			ixx="0.04"
 			ixy="0"
 			ixz="0"
-			iyy="0.104167"
+			iyy="0.04"
 			iyz="0"
-			izz="0.254167"
+			izz="0.08"
 		/>
 	</inertial>
@@ -549,6 +549,6 @@
        <update_rate>10</update_rate>
        <grip_count_threshold>4</grip_count_threshold>
-       <max_grip_count>30</max_grip_count>
-       <release_tolerance>0.01</release_tolerance>
+       <max_grip_count>8</max_grip_count>
+       <release_tolerance>0.001</release_tolerance>
        <disable_collisions_on_attach>false</disable_collisions_on_attach>
        <contact_topic>__default_topic__</contact_topic>

File: demo_navi/src/urdf/xacro/rim.urdf.xacro (robot description, xacro)
@@ -10,5 +10,5 @@
 			<inertial>
 				<origin xyz="0 0 0"/>
-				<mass value="1"/>
+				<mass value="2.5"/>
 				<inertia
 					ixx="0.000007"
@@ -45,6 +45,5 @@
 				rpy="${rpy}"
 			/>
-			<limit effort="100000" velocity="100000"/>
-			<joint_properties friction="1.0"/>
+			<limit effort="1000000000" velocity="1000"/>
 		</joint>
 		<xacro:roller_macro
@@ -95,8 +94,8 @@
 		</transmission>
 		<gazebo reference = "rim_${name}_link">
-  				<mu1>50.0</mu1>
-  				<mu2>25.0</mu2>
-  				<selfCollide>False</selfCollide>
+  				<!--<mu1>50.0</mu1>
+  				<mu2>25.0</mu2>-->
       			<!--kp  value="10000000.0" />
+      			<selfCollide>False</selfCollide>
       			<kd  value="10000000.0" />
       			<dampingFactor>10</dampingFactor>

File: demo_navi/src/urdf/xacro/roller.urdf.xacro (robot description, xacro)
@@ -7,5 +7,5 @@
 		<link name="roller_${name}_rim_${parent}_link">
 			<inertial>
-				<mass value="0.1"/>
+				<mass value="1"/>
 				<inertia
 					ixx="6.008e-07"
@@ -42,10 +42,9 @@
 				rpy="${rpy}"
 			/>
-			<limit effort="100000000" velocity="1000000000"/>
-			<joint_properties friction="1.0"/>
+			<limit effort="100000000" velocity="1000"/>
 		</joint>
 	<gazebo reference="roller_${name}_rim_${parent}_link">
-  			<mu1>50.0</mu1>
-  			<mu2>25.0</mu2>
+  			<!--<mu1>50.0</mu1>
+  			<mu2>25.0</mu2>-->
       		<kp  value="10000000000.0" />
       		<kd  value="10000000000.0" />
@@ -54,6 +53,6 @@
     <material>Gazebo/Grey</material>
   </gazebo>
-  <selfCollide>False</selfCollide>
   <!--<gazebo reference="roller_${name}_rim_${parent}_joint">
+    <selfCollide>False</selfCollide>
     <dampingFactor>10</dampingFactor>
     <minDepth>0.001</minDepth>
