Commit message: Updated stability

File: demo_navi/src/urdf/model.urdf.xacro (robot description, xacro)
@@ -228,6 +228,6 @@
     <inertial>
       <origin rpy="0 0 0" xyz="-0.147 0 0.05"/>
-      <mass value="5"/>
-      <inertia ixx="0.04" ixy="0" ixz="0" iyy="0.04" iyz="0" izz="0.08"/>
+      <mass value="15"/>
+      <inertia ixx="0.15" ixy="0" ixz="0" iyy="0.104167" iyz="0" izz="0.254167"/>
     </inertial>
     <visual>
@@ -260,6 +260,6 @@
     <inertial>
       <origin xyz="0 0 0"/>
-      <mass value="2.5"/>
-      <inertia ixx="0.000007" ixy="0" ixz="0" iyy="0.000007" iyz="0" izz="0.000008"/>
+      <mass value="0.5"/>
+      <inertia ixx="0.0007" ixy="0" ixz="0" iyy="0.0007" iyz="0" izz="0.0008"/>
     </inertial>
     <visual>
@@ -286,6 +286,6 @@
   <link name="roller_s_rim_left_link">
     <inertial>
-      <mass value="1"/>
-      <inertia ixx="6.008e-07" ixy="0" ixz="0" iyy="6.008e-07" iyz="0" izz="0.0000000101"/>
+      <mass value="0.1"/>
+      <inertia ixx="6.8e-03" ixy="0" ixz="0" iyy="6.8e-03" iyz="0" izz="0.000101"/>
     </inertial>
     <visual>
@@ -312,9 +312,9 @@
   <gazebo reference="roller_s_rim_left_link">
     <!--<mu1>50.0</mu1>
-  			<mu2>25.0</mu2>-->
-    <kp value="10000000000.0"/>
-    <kd value="10000000000.0"/>
-    <dampingFactor>10</dampingFactor>
-    <minDepth>0.001</minDepth>
+  			<mu2>25.0</mu2>
+      		<kp  value="10000000000.0" />
+      		<kd  value="10000000000.0" /-->
+    <dampingFactor>10</dampingFactor>
+    <minDepth>1</minDepth>
     <material>Gazebo/Grey</material>
   </gazebo>
@@ -326,6 +326,6 @@
   <link name="roller_nw_rim_left_link">
     <inertial>
-      <mass value="1"/>
-      <inertia ixx="6.008e-07" ixy="0" ixz="0" iyy="6.008e-07" iyz="0" izz="0.0000000101"/>
+      <mass value="0.1"/>
+      <inertia ixx="6.8e-03" ixy="0" ixz="0" iyy="6.8e-03" iyz="0" izz="0.000101"/>
     </inertial>
     <visual>
@@ -352,9 +352,9 @@
   <gazebo reference="roller_nw_rim_left_link">
     <!--<mu1>50.0</mu1>
-  			<mu2>25.0</mu2>-->
-    <kp value="10000000000.0"/>
-    <kd value="10000000000.0"/>
-    <dampingFactor>10</dampingFactor>
-    <minDepth>0.001</minDepth>
+  			<mu2>25.0</mu2>
+      		<kp  value="10000000000.0" />
+      		<kd  value="10000000000.0" /-->
+    <dampingFactor>10</dampingFactor>
+    <minDepth>1</minDepth>
     <material>Gazebo/Grey</material>
   </gazebo>
@@ -366,6 +366,6 @@
   <link name="roller_ne_rim_left_link">
     <inertial>
-      <mass value="1"/>
-      <inertia ixx="6.008e-07" ixy="0" ixz="0" iyy="6.008e-07" iyz="0" izz="0.0000000101"/>
+      <mass value="0.1"/>
+      <inertia ixx="6.8e-03" ixy="0" ixz="0" iyy="6.8e-03" iyz="0" izz="0.000101"/>
     </inertial>
     <visual>
@@ -392,9 +392,9 @@
   <gazebo reference="roller_ne_rim_left_link">
     <!--<mu1>50.0</mu1>
-  			<mu2>25.0</mu2>-->
-    <kp value="10000000000.0"/>
-    <kd value="10000000000.0"/>
-    <dampingFactor>10</dampingFactor>
-    <minDepth>0.001</minDepth>
+  			<mu2>25.0</mu2>
+      		<kp  value="10000000000.0" />
+      		<kd  value="10000000000.0" /-->
+    <dampingFactor>10</dampingFactor>
+    <minDepth>1</minDepth>
     <material>Gazebo/Grey</material>
   </gazebo>
@@ -406,6 +406,6 @@
   <link name="roller_sw_rim_left_link">
     <inertial>
-      <mass value="1"/>
-      <inertia ixx="6.008e-07" ixy="0" ixz="0" iyy="6.008e-07" iyz="0" izz="0.0000000101"/>
+      <mass value="0.1"/>
+      <inertia ixx="6.8e-03" ixy="0" ixz="0" iyy="6.8e-03" iyz="0" izz="0.000101"/>
     </inertial>
     <visual>
@@ -432,9 +432,9 @@
   <gazebo reference="roller_sw_rim_left_link">
     <!--<mu1>50.0</mu1>
-  			<mu2>25.0</mu2>-->
-    <kp value="10000000000.0"/>
-    <kd value="10000000000.0"/>
-    <dampingFactor>10</dampingFactor>
-    <minDepth>0.001</minDepth>
+  			<mu2>25.0</mu2>
+      		<kp  value="10000000000.0" />
+      		<kd  value="10000000000.0" /-->
+    <dampingFactor>10</dampingFactor>
+    <minDepth>1</minDepth>
     <material>Gazebo/Grey</material>
   </gazebo>
@@ -446,6 +446,6 @@
   <link name="roller_n_rim_left_link">
     <inertial>
-      <mass value="1"/>
-      <inertia ixx="6.008e-07" ixy="0" ixz="0" iyy="6.008e-07" iyz="0" izz="0.0000000101"/>
+      <mass value="0.1"/>
+      <inertia ixx="6.8e-03" ixy="0" ixz="0" iyy="6.8e-03" iyz="0" izz="0.000101"/>
     </inertial>
     <visual>
@@ -472,9 +472,9 @@
   <gazebo reference="roller_n_rim_left_link">
     <!--<mu1>50.0</mu1>
-  			<mu2>25.0</mu2>-->
-    <kp value="10000000000.0"/>
-    <kd value="10000000000.0"/>
-    <dampingFactor>10</dampingFactor>
-    <minDepth>0.001</minDepth>
+  			<mu2>25.0</mu2>
+      		<kp  value="10000000000.0" />
+      		<kd  value="10000000000.0" /-->
+    <dampingFactor>10</dampingFactor>
+    <minDepth>1</minDepth>
     <material>Gazebo/Grey</material>
   </gazebo>
@@ -486,6 +486,6 @@
   <link name="roller_se_rim_left_link">
     <inertial>
-      <mass value="1"/>
-      <inertia ixx="6.008e-07" ixy="0" ixz="0" iyy="6.008e-07" iyz="0" izz="0.0000000101"/>
+      <mass value="0.1"/>
+      <inertia ixx="6.8e-03" ixy="0" ixz="0" iyy="6.8e-03" iyz="0" izz="0.000101"/>
     </inertial>
     <visual>
@@ -512,9 +512,9 @@
   <gazebo reference="roller_se_rim_left_link">
     <!--<mu1>50.0</mu1>
-  			<mu2>25.0</mu2>-->
-    <kp value="10000000000.0"/>
-    <kd value="10000000000.0"/>
-    <dampingFactor>10</dampingFactor>
-    <minDepth>0.001</minDepth>
+  			<mu2>25.0</mu2>
+      		<kp  value="10000000000.0" />
+      		<kd  value="10000000000.0" /-->
+    <dampingFactor>10</dampingFactor>
+    <minDepth>1</minDepth>
     <material>Gazebo/Grey</material>
   </gazebo>
@@ -535,17 +535,17 @@
   </transmission>
   <gazebo reference="rim_left_link">
-    <!--<mu1>50.0</mu1>
-  				<mu2>25.0</mu2>-->
+    <!--mu1>50.0</mu1>
+  				<mu2>25.0</mu2-->
     <!--kp  value="10000000.0" />
       			<selfCollide>False</selfCollide>
-      			<kd  value="10000000.0" />
-      			<dampingFactor>10</dampingFactor>
-				<minDepth>0.001</minDepth-->
+      			<kd  value="10000000.0" /-->
+    <dampingFactor>10</dampingFactor>
+    <minDepth>1</minDepth>
   </gazebo>
   <link name="rim_back_link">
     <inertial>
       <origin xyz="0 0 0"/>
-      <mass value="2.5"/>
-      <inertia ixx="0.000007" ixy="0" ixz="0" iyy="0.000007" iyz="0" izz="0.000008"/>
+      <mass value="0.5"/>
+      <inertia ixx="0.0007" ixy="0" ixz="0" iyy="0.0007" iyz="0" izz="0.0008"/>
     </inertial>
     <visual>
@@ -572,6 +572,6 @@
   <link name="roller_s_rim_back_link">
     <inertial>
-      <mass value="1"/>
-      <inertia ixx="6.008e-07" ixy="0" ixz="0" iyy="6.008e-07" iyz="0" izz="0.0000000101"/>
+      <mass value="0.1"/>
+      <inertia ixx="6.8e-03" ixy="0" ixz="0" iyy="6.8e-03" iyz="0" izz="0.000101"/>
     </inertial>
     <visual>
@@ -598,9 +598,9 @@
   <gazebo reference="roller_s_rim_back_link">
     <!--<mu1>50.0</mu1>
-  			<mu2>25.0</mu2>-->
-    <kp value="10000000000.0"/>
-    <kd value="10000000000.0"/>
-    <dampingFactor>10</dampingFactor>
-    <minDepth>0.001</minDepth>
+  			<mu2>25.0</mu2>
+      		<kp  value="10000000000.0" />
+      		<kd  value="10000000000.0" /-->
+    <dampingFactor>10</dampingFactor>
+    <minDepth>1</minDepth>
     <material>Gazebo/Grey</material>
   </gazebo>
@@ -612,6 +612,6 @@
   <link name="roller_nw_rim_back_link">
     <inertial>
-      <mass value="1"/>
-      <inertia ixx="6.008e-07" ixy="0" ixz="0" iyy="6.008e-07" iyz="0" izz="0.0000000101"/>
+      <mass value="0.1"/>
+      <inertia ixx="6.8e-03" ixy="0" ixz="0" iyy="6.8e-03" iyz="0" izz="0.000101"/>
     </inertial>
     <visual>
@@ -638,9 +638,9 @@
   <gazebo reference="roller_nw_rim_back_link">
     <!--<mu1>50.0</mu1>
-  			<mu2>25.0</mu2>-->
-    <kp value="10000000000.0"/>
-    <kd value="10000000000.0"/>
-    <dampingFactor>10</dampingFactor>
-    <minDepth>0.001</minDepth>
+  			<mu2>25.0</mu2>
+      		<kp  value="10000000000.0" />
+      		<kd  value="10000000000.0" /-->
+    <dampingFactor>10</dampingFactor>
+    <minDepth>1</minDepth>
     <material>Gazebo/Grey</material>
   </gazebo>
@@ -652,6 +652,6 @@
   <link name="roller_ne_rim_back_link">
     <inertial>
-      <mass value="1"/>
-      <inertia ixx="6.008e-07" ixy="0" ixz="0" iyy="6.008e-07" iyz="0" izz="0.0000000101"/>
+      <mass value="0.1"/>
+      <inertia ixx="6.8e-03" ixy="0" ixz="0" iyy="6.8e-03" iyz="0" izz="0.000101"/>
     </inertial>
     <visual>
@@ -678,9 +678,9 @@
   <gazebo reference="roller_ne_rim_back_link">
     <!--<mu1>50.0</mu1>
-  			<mu2>25.0</mu2>-->
-    <kp value="10000000000.0"/>
-    <kd value="10000000000.0"/>
-    <dampingFactor>10</dampingFactor>
-    <minDepth>0.001</minDepth>
+  			<mu2>25.0</mu2>
+      		<kp  value="10000000000.0" />
+      		<kd  value="10000000000.0" /-->
+    <dampingFactor>10</dampingFactor>
+    <minDepth>1</minDepth>
     <material>Gazebo/Grey</material>
   </gazebo>
@@ -692,6 +692,6 @@
   <link name="roller_sw_rim_back_link">
     <inertial>
-      <mass value="1"/>
-      <inertia ixx="6.008e-07" ixy="0" ixz="0" iyy="6.008e-07" iyz="0" izz="0.0000000101"/>
+      <mass value="0.1"/>
+      <inertia ixx="6.8e-03" ixy="0" ixz="0" iyy="6.8e-03" iyz="0" izz="0.000101"/>
     </inertial>
     <visual>
@@ -718,9 +718,9 @@
   <gazebo reference="roller_sw_rim_back_link">
     <!--<mu1>50.0</mu1>
-  			<mu2>25.0</mu2>-->
-    <kp value="10000000000.0"/>
-    <kd value="10000000000.0"/>
-    <dampingFactor>10</dampingFactor>
-    <minDepth>0.001</minDepth>
+  			<mu2>25.0</mu2>
+      		<kp  value="10000000000.0" />
+      		<kd  value="10000000000.0" /-->
+    <dampingFactor>10</dampingFactor>
+    <minDepth>1</minDepth>
     <material>Gazebo/Grey</material>
   </gazebo>
@@ -732,6 +732,6 @@
   <link name="roller_n_rim_back_link">
     <inertial>
-      <mass value="1"/>
-      <inertia ixx="6.008e-07" ixy="0" ixz="0" iyy="6.008e-07" iyz="0" izz="0.0000000101"/>
+      <mass value="0.1"/>
+      <inertia ixx="6.8e-03" ixy="0" ixz="0" iyy="6.8e-03" iyz="0" izz="0.000101"/>
     </inertial>
     <visual>
@@ -758,9 +758,9 @@
   <gazebo reference="roller_n_rim_back_link">
     <!--<mu1>50.0</mu1>
-  			<mu2>25.0</mu2>-->
-    <kp value="10000000000.0"/>
-    <kd value="10000000000.0"/>
-    <dampingFactor>10</dampingFactor>
-    <minDepth>0.001</minDepth>
+  			<mu2>25.0</mu2>
+      		<kp  value="10000000000.0" />
+      		<kd  value="10000000000.0" /-->
+    <dampingFactor>10</dampingFactor>
+    <minDepth>1</minDepth>
     <material>Gazebo/Grey</material>
   </gazebo>
@@ -772,6 +772,6 @@
   <link name="roller_se_rim_back_link">
     <inertial>
-      <mass value="1"/>
-      <inertia ixx="6.008e-07" ixy="0" ixz="0" iyy="6.008e-07" iyz="0" izz="0.0000000101"/>
+      <mass value="0.1"/>
+      <inertia ixx="6.8e-03" ixy="0" ixz="0" iyy="6.8e-03" iyz="0" izz="0.000101"/>
     </inertial>
     <visual>
@@ -798,9 +798,9 @@
   <gazebo reference="roller_se_rim_back_link">
     <!--<mu1>50.0</mu1>
-  			<mu2>25.0</mu2>-->
-    <kp value="10000000000.0"/>
-    <kd value="10000000000.0"/>
-    <dampingFactor>10</dampingFactor>
-    <minDepth>0.001</minDepth>
+  			<mu2>25.0</mu2>
+      		<kp  value="10000000000.0" />
+      		<kd  value="10000000000.0" /-->
+    <dampingFactor>10</dampingFactor>
+    <minDepth>1</minDepth>
     <material>Gazebo/Grey</material>
   </gazebo>
@@ -821,17 +821,17 @@
   </transmission>
   <gazebo reference="rim_back_link">
-    <!--<mu1>50.0</mu1>
-  				<mu2>25.0</mu2>-->
+    <!--mu1>50.0</mu1>
+  				<mu2>25.0</mu2-->
     <!--kp  value="10000000.0" />
       			<selfCollide>False</selfCollide>
-      			<kd  value="10000000.0" />
-      			<dampingFactor>10</dampingFactor>
-				<minDepth>0.001</minDepth-->
+      			<kd  value="10000000.0" /-->
+    <dampingFactor>10</dampingFactor>
+    <minDepth>1</minDepth>
   </gazebo>
   <link name="rim_right_link">
     <inertial>
       <origin xyz="0 0 0"/>
-      <mass value="2.5"/>
-      <inertia ixx="0.000007" ixy="0" ixz="0" iyy="0.000007" iyz="0" izz="0.000008"/>
+      <mass value="0.5"/>
+      <inertia ixx="0.0007" ixy="0" ixz="0" iyy="0.0007" iyz="0" izz="0.0008"/>
     </inertial>
     <visual>
@@ -858,6 +858,6 @@
   <link name="roller_s_rim_right_link">
     <inertial>
-      <mass value="1"/>
-      <inertia ixx="6.008e-07" ixy="0" ixz="0" iyy="6.008e-07" iyz="0" izz="0.0000000101"/>
+      <mass value="0.1"/>
+      <inertia ixx="6.8e-03" ixy="0" ixz="0" iyy="6.8e-03" iyz="0" izz="0.000101"/>
     </inertial>
     <visual>
@@ -884,9 +884,9 @@
   <gazebo reference="roller_s_rim_right_link">
     <!--<mu1>50.0</mu1>
-  			<mu2>25.0</mu2>-->
-    <kp value="10000000000.0"/>
-    <kd value="10000000000.0"/>
-    <dampingFactor>10</dampingFactor>
-    <minDepth>0.001</minDepth>
+  			<mu2>25.0</mu2>
+      		<kp  value="10000000000.0" />
+      		<kd  value="10000000000.0" /-->
+    <dampingFactor>10</dampingFactor>
+    <minDepth>1</minDepth>
     <material>Gazebo/Grey</material>
   </gazebo>
@@ -898,6 +898,6 @@
   <link name="roller_nw_rim_right_link">
     <inertial>
-      <mass value="1"/>
-      <inertia ixx="6.008e-07" ixy="0" ixz="0" iyy="6.008e-07" iyz="0" izz="0.0000000101"/>
+      <mass value="0.1"/>
+      <inertia ixx="6.8e-03" ixy="0" ixz="0" iyy="6.8e-03" iyz="0" izz="0.000101"/>
     </inertial>
     <visual>
@@ -924,9 +924,9 @@
   <gazebo reference="roller_nw_rim_right_link">
     <!--<mu1>50.0</mu1>
-  			<mu2>25.0</mu2>-->
-    <kp value="10000000000.0"/>
-    <kd value="10000000000.0"/>
-    <dampingFactor>10</dampingFactor>
-    <minDepth>0.001</minDepth>
+  			<mu2>25.0</mu2>
+      		<kp  value="10000000000.0" />
+      		<kd  value="10000000000.0" /-->
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
File: demo_navi/src/urdf/xacro/main.urdf.xacro (robot description, xacro)
@@ -4,5 +4,5 @@
   name="demo_DIR"
 >
-	<xacro:include filename="$(find demo_navi)/src/urdf/xacro/rim.urdf.xacro"/>
+  <xacro:include filename="$(find demo_navi)/src/urdf/xacro/rim.urdf.xacro"/>
   <xacro:include filename="$(find demo_navi)/src/urdf/xacro/common_materials.xacro" />
   <xacro:include filename="$(find realsense2_description)/urdf/_d435.urdf.xacro" />
@@ -16,12 +16,12 @@
 		<origin xyz="-0.147 0 0.05"
 			rpy="0 0 0" />
-		<mass value="5"/>
+		<mass value="15"/>
 		<inertia
-			ixx="0.04"
+			ixx="0.15"
 			ixy="0"
 			ixz="0"
-			iyy="0.04"
+			iyy="0.104167"
 			iyz="0"
-			izz="0.08"
+			izz="0.254167"
 		/>
 	</inertial>
@@ -151,6 +151,6 @@
          <inertial>
           <origin xyz="0 0 0" rpy="0 0 0" />
-            <mass value="0.001" />
-            <inertia ixx="0.001" ixy="0.0" ixz="0.0" iyy="0.001" iyz="0.0" izz="0.001" />
+            <mass value="0.1" />
+            <inertia ixx="0.01" ixy="0.0" ixz="0.0" iyy="0.01" iyz="0.0" izz="0.01"/>
          </inertial>
       </link>
@@ -171,6 +171,6 @@
          <inertial>
           <origin xyz="0.04825 0 0.14" rpy="0 0 0" />
-            <mass value="0.001" />
-            <inertia ixx="0.001" ixy="0.0" ixz="0.0" iyy="0.001" iyz="0.0" izz="0.001" />
+            <mass value="0.1" />
+           <inertia ixx="0.01" ixy="0.0" ixz="0.0" iyy="0.01" iyz="0.0" izz="0.01"/>
          </inertial>
       </link>
@@ -191,6 +191,6 @@
          <inertial>
           <origin xyz="0 0 0.14203" rpy="0 0 0" />
-            <mass value="0.001" />
-            <inertia ixx="0.001" ixy="0.0" ixz="0.0" iyy="0.001" iyz="0.0" izz="0.001"/>
+            <mass value="0.1" />
+            <inertia ixx="0.01" ixy="0.0" ixz="0.0" iyy="0.01" iyz="0.0" izz="0.01"/>
          </inertial>
       </link>
@@ -211,6 +211,6 @@
          <inertial>
           <origin xyz="0 0 0" rpy="0 0 0" />
-            <mass value="0.001" />
-            <inertia ixx="0.001" ixy="0.0" ixz="0.0" iyy="0.001" iyz="0.0" izz="0.001" />
+            <mass value="0.1" />
+            <inertia ixx="0.01" ixy="0.0" ixz="0.0" iyy="0.01" iyz="0.0" izz="0.01"/>
          </inertial>
       </link>
@@ -231,6 +231,6 @@
          <inertial>
           <origin xyz="0 0 0.043" rpy="0 0 0" />
-            <mass value="0.001" />
-            <inertia ixx="0.001" ixy="0.0" ixz="0.0" iyy="0.001" iyz="0.0" izz="0.001" />
+            <mass value="0.1" />
+            <inertia ixx="0.01" ixy="0.0" ixz="0.0" iyy="0.01" iyz="0.0" izz="0.01"/>
          </inertial>
       </link>
@@ -251,6 +251,6 @@
          <inertial>
           <origin xyz = "0 0 0" rpy="0 0 1.57" />
-            <mass value="0.001" />
-            <inertia ixx="0.001" ixy="0.0" ixz="0.0" iyy="0.001" iyz="0.0" izz="0.001" />
+            <mass value="0.1" />
+            <inertia ixx="0.01" ixy="0.0" ixz="0.0" iyy="0.01" iyz="0.0" izz="0.01"/>
          </inertial>
       </link>
@@ -273,6 +273,6 @@
          <inertial>
           <origin xyz="0 -0.0007 0" rpy="0 0 1.57" />
-            <mass value="0.001" />
-            <inertia ixx="0.001" ixy="0.0" ixz="0.0" iyy="0.001" iyz="0.0" izz="0.001" />
+            <mass value="0.1" />
+            <inertia ixx="0.01" ixy="0.0" ixz="0.0" iyy="0.01" iyz="0.0" izz="0.01"/>
          </inertial>
       </link>
@@ -293,6 +293,6 @@
          <inertial>
           <origin xyz="0 0.0007 0" rpy="0 0 -1.57" />
-            <mass value="0.001" />
-            <inertia ixx="0.001" ixy="0.0" ixz="0.0" iyy="0.001" iyz="0.0" izz="0.001" />
+            <mass value="0.1" />
+            <inertia ixx="0.01" ixy="0.0" ixz="0.0" iyy="0.01" iyz="0.0" izz="0.01"/>
          </inertial>
       </link>
@@ -303,5 +303,5 @@
          <child link="shoulder_link" />
          <axis xyz="0 0 1" />
-         <limit lower="-3.1415" upper="3.1415" effort="100" velocity="0.785" />
+         <limit lower="-3.1415" upper="3.1415" effort="100" velocity="1.571" />
       </joint>
       <joint name="joint_2" type="revolute">
@@ -462,5 +462,5 @@
       <update_rate>100</update_rate>
       <visualize>true</visualize>
-      <topic>__default_topic__</topic>
+      <topic>__default_topic_imu_link__</topic>
       <plugin filename="libgazebo_ros_imu_sensor.so" name="imu_plugin">
         <topicName>imu</topicName>

File: demo_navi/src/urdf/xacro/rim.urdf.xacro (robot description, xacro)
@@ -10,12 +10,12 @@
 			<inertial>
 				<origin xyz="0 0 0"/>
-				<mass value="2.5"/>
+				<mass value="0.5"/>
 				<inertia
-					ixx="0.000007"
+					ixx="0.0007"
 					ixy="0"
 					ixz="0"
-					iyy="0.000007"
+					iyy="0.0007"
 					iyz="0"
-					izz="0.000008"
+					izz="0.0008"
 				/>
 			</inertial>
@@ -94,11 +94,11 @@
 		</transmission>
 		<gazebo reference = "rim_${name}_link">
-  				<!--<mu1>50.0</mu1>
-  				<mu2>25.0</mu2>-->
+  				<!--mu1>50.0</mu1>
+  				<mu2>25.0</mu2-->
       			<!--kp  value="10000000.0" />
       			<selfCollide>False</selfCollide>
-      			<kd  value="10000000.0" />
+      			<kd  value="10000000.0" /-->
       			<dampingFactor>10</dampingFactor>
-				<minDepth>0.001</minDepth-->
+				<minDepth>1</minDepth>
 		</gazebo>
 	</xacro:macro>

File: demo_navi/src/urdf/xacro/roller.urdf.xacro (robot description, xacro)
@@ -7,12 +7,12 @@
 		<link name="roller_${name}_rim_${parent}_link">
 			<inertial>
-				<mass value="1"/>
+				<mass value="0.1"/>
 				<inertia
-					ixx="6.008e-07"
+					ixx="6.8e-03"
 					ixy="0"
 					ixz="0"
-					iyy="6.008e-07"
+					iyy="6.8e-03"
 					iyz="0"
-					izz="0.0000000101"
+					izz="0.000101"
 				/>
 			</inertial>
@@ -46,9 +46,9 @@
 	<gazebo reference="roller_${name}_rim_${parent}_link">
   			<!--<mu1>50.0</mu1>
-  			<mu2>25.0</mu2>-->
+  			<mu2>25.0</mu2>
       		<kp  value="10000000000.0" />
-      		<kd  value="10000000000.0" />
+      		<kd  value="10000000000.0" /-->
     	  	<dampingFactor>10</dampingFactor>
-    		<minDepth>0.001</minDepth>
+    		<minDepth>1</minDepth>
     <material>Gazebo/Grey</material>
   </gazebo>

Commit message: Updated 0406

File: demo_navi/src/urdf/model.urdf.xacro (robot description, xacro)
@@ -1604,5 +1604,5 @@
       <grip_count_threshold>4</grip_count_threshold>
       <max_grip_count>8</max_grip_count>
-      <release_tolerance>0.001</release_tolerance>
+      <release_tolerance>0.01</release_tolerance>
       <disable_collisions_on_attach>false</disable_collisions_on_attach>
       <contact_topic>__default_topic__</contact_topic>

File: demo_navi/src/urdf/xacro/main.urdf.xacro (robot description, xacro)
@@ -353,5 +353,5 @@
          <child link="gripper_1_link" />
          <axis xyz="0 -1 0" />
-         <limit lower="0" upper="0.027" effort="100" velocity="0.5" />
+         <limit lower="0" upper="0.027" effort="1000" velocity="0.5" />
       </joint>
       <joint name="gripper_prismatic_joint_2" type="prismatic">
@@ -360,5 +360,5 @@
          <child link="gripper_2_link" />
          <axis xyz="0 1 0" />
-         <limit lower="0" upper="0.027" effort="100" velocity="0.5" />
+         <limit lower="0" upper="0.027" effort="1000" velocity="0.5" />
       </joint>
   <transmission name="tran1">
@@ -547,8 +547,8 @@
         </arm>
        <forces_angle_tolerance>100</forces_angle_tolerance>
-       <update_rate>10</update_rate>
+       <update_rate>4</update_rate>
        <grip_count_threshold>4</grip_count_threshold>
        <max_grip_count>8</max_grip_count>
-       <release_tolerance>0.001</release_tolerance>
+       <release_tolerance>0.007</release_tolerance>
        <disable_collisions_on_attach>false</disable_collisions_on_attach>
        <contact_topic>__default_topic__</contact_topic>
@@ -567,3 +567,13 @@
     		<material>Gazebo/Black</material>
   	</gazebo>
+  	<gazebo reference="gripper_1_link">
+    		<mu1>5.5</mu1>
+  		<mu2>5.5</mu2>
+		<dampingFactor>10</dampingFactor>
+  	</gazebo>
+  	<gazebo reference="gripper_2_link">
+    		<mu1>5.5</mu1>
+  		<mu2>5.5</mu2>
+  		<dampingFactor>10</dampingFactor>
+  	</gazebo>
 </robot>
