Commit message: Added robocup_ objects

File: demo_navi/src/urdf/xacro/rim.urdf.xacro (robot description, xacro)
@@ -12,10 +12,10 @@
 				<mass value="0.5"/>
 				<inertia
-					ixx="0.0007"
+					ixx="0.7"
 					ixy="0"
 					ixz="0"
-					iyy="0.0007"
+					iyy="0.7"
 					iyz="0"
-					izz="0.0008"
+					izz="0.8"
 				/>
 			</inertial>
@@ -45,5 +45,5 @@
 				rpy="${rpy}"
 			/>
-			<limit effort="1000000000" velocity="1000"/>
+			<limit effort="100000000" velocity="10"/>
 		</joint>
 		<xacro:roller_macro

File: demo_navi/src/urdf/xacro/roller.urdf.xacro (robot description, xacro)
@@ -9,10 +9,10 @@
 				<mass value="0.1"/>
 				<inertia
-					ixx="6.8e-03"
+					ixx="6.8e-01"
 					ixy="0"
 					ixz="0"
-					iyy="6.8e-03"
+					iyy="6.8e-01"
 					iyz="0"
-					izz="0.000101"
+					izz="0.0101"
 				/>
 			</inertial>
@@ -42,5 +42,5 @@
 				rpy="${rpy}"
 			/>
-			<limit effort="100000000" velocity="1000"/>
+			<limit effort="100000000" velocity="10"/>
 		</joint>
 	<gazebo reference="roller_${name}_rim_${parent}_link">
