Commit message: add_controllers

File: demo_navi/src/urdf/xacro/main.urdf.xacro (robot description, xacro)
@@ -57,5 +57,5 @@
 	<xacro:rim_macro
 		name="back"
-		color="0 0.3 0"
+		color="0.3 0 0"
 		xyz="-0.397 0 0.04"
 		rpy="1.570796326794896 0 1.5708"
@@ -63,5 +63,5 @@
 	<xacro:rim_macro
 		name="right"
-		color="0 0 0.3"
+		color="0.3 0 0"
 		xyz="-0.03 -0.208 0.04"
 		rpy="1.570796326794896 0 -2.61799"
@@ -180,5 +180,5 @@
       <update_rate>15.0</update_rate>
       <pose>0 0 0 0 0 0</pose>
-      <visualize>true</visualize>
+      <visualize>false</visualize>
       <ray>
         <scan>

File: demo_navi/src/urdf/xacro/rim.urdf.xacro (robot description, xacro)
@@ -32,4 +32,12 @@
 					<mesh filename="package://demo_navi/src/meshes/rim.stl"/>
 				</geometry>
+				<surface>
+        			<friction>
+          				<ode>
+            				<mu>0.5</mu>
+            				<mu2>0.5</mu2>
+          				</ode>
+        			</friction>
+      			</surface>
 			</collision>
 		</link>
@@ -45,4 +53,6 @@
 				rpy="${rpy}"
 			/>
+			<limit effort="100000" velocity="100000"/>
+			<joint_properties friction="1.0"/>
 		</joint>
 		<xacro:roller_macro
@@ -85,8 +95,8 @@
 			<type>transmission_interface/SimpleTransmission</type>
 			<joint name="rim_${name}_joint">
-				<hardwareInterface>hardware_interface/VelocityJointInterface</hardwareInterface>
+				<hardwareInterface>hardware_interface/EffortJointInterface</hardwareInterface>
 			</joint>
 			<actuator name="rim_${name}_motor">
-				<hardwareInterface>hardware_interface/VelocityJointInterface</hardwareInterface>
+				<hardwareInterface>hardware_interface/EffortJointInterface</hardwareInterface>
 				<mechanicalReduction>1</mechanicalReduction>
 			</actuator>
@@ -96,4 +106,8 @@
 			<minDepth>0.001</minDepth>
 		</gazebo>
+		<gazebo reference = "rim_${name}_joint">
+			<dampingFactor>10</dampingFactor>
+			<minDepth>0.001</minDepth>
+		</gazebo>
 	</xacro:macro>
 </robot>

File: demo_navi/src/urdf/xacro/roller.urdf.xacro (robot description, xacro)
@@ -7,12 +7,12 @@
 		<link name="roller_${name}_rim_${parent}_link">
 			<inertial>
-				<mass value="0.00113845"/>
+				<mass value="0.5"/>
 				<inertia
-					ixx="2.0308e-05"
+					ixx="8.8445e-06"
 					ixy="0"
 					ixz="0"
-					iyy="1.0512e-05"
+					iyy="8.8445e-06"
 					iyz="0"
-					izz="2.0308e-05"
+					izz="3.627e-04"
 				/>
 			</inertial>
@@ -29,4 +29,12 @@
 					<mesh filename="package://demo_navi/src/meshes/roller.stl"/>
 				</geometry>
+				<surface>
+        			<friction>
+          				<ode>
+            				<mu>0.5</mu>
+            				<mu2>0.5</mu2>
+          				</ode>
+        			</friction>
+      			</surface>
 			</collision>
 		</link>
@@ -42,4 +50,6 @@
 				rpy="${rpy}"
 			/>
+			<limit effort="10000000" velocity="1000000"/>
+			<joint_properties friction="1.0"/>
 		</joint>
 	<gazebo reference = "roller_${name}_rim_${parent}_link">
@@ -47,4 +57,8 @@
 		<minDepth>0.001</minDepth>
 	</gazebo>
+	<gazebo reference = "roller_${name}_rim_${parent}_joint">
+		<dampingFactor>10</dampingFactor>
+		<minDepth>0.001</minDepth>
+	</gazebo>
 	</xacro:macro>
 </robot>

Commit message: Updated arm

File: demo_navi/src/urdf/xacro/main.urdf.xacro (robot description, xacro)
@@ -120,5 +120,5 @@
     </link>
     <!--WIDOWXL ARM LINKS & JOINTS-->
-          <link name="shoulder_link">
+        <link name="shoulder_link">
          <visual>
           <origin xyz="0 0 0" rpy="0 0 0" />
@@ -136,6 +136,6 @@
          <inertial>
           <origin xyz="0 0 0" rpy="0 0 0" />
-            <mass value="0.1" />
-            <inertia ixx="0.1" ixy="0.0" ixz="0.0" iyy="0.1" iyz="0.0" izz="0.1" />
+            <mass value="0.01" />
+            <inertia ixx="0.01" ixy="0.0" ixz="0.0" iyy="0.01" iyz="0.0" izz="0.01" />
          </inertial>
       </link>
@@ -156,6 +156,6 @@
          <inertial>
           <origin xyz="0.04825 0 0.14" rpy="0 0 0" />
-            <mass value="0.1" />
-            <inertia ixx="0.1" ixy="0.0" ixz="0.0" iyy="0.1" iyz="0.0" izz="0.1" />
+            <mass value="0.01" />
+            <inertia ixx="0.01" ixy="0.0" ixz="0.0" iyy="0.01" iyz="0.0" izz="0.01" />
          </inertial>
       </link>
@@ -176,6 +176,6 @@
          <inertial>
           <origin xyz="0 0 0.14203" rpy="0 0 0" />
-            <mass value="0.1" />
-            <inertia ixx="1.0" ixy="0.0" ixz="0.0" iyy="1.0" iyz="0.0" izz="1.0"/>
+            <mass value="0.01" />
+            <inertia ixx="0.01" ixy="0.0" ixz="0.0" iyy="0.01" iyz="0.0" izz="0.01"/>
          </inertial>
       </link>
@@ -196,6 +196,6 @@
          <inertial>
           <origin xyz="0 0 0" rpy="0 0 0" />
-            <mass value="0.1" />
-            <inertia ixx="0.1" ixy="0.0" ixz="0.0" iyy="0.1" iyz="0.0" izz="0.1" />
+            <mass value="0.01" />
+            <inertia ixx="0.01" ixy="0.0" ixz="0.0" iyy="0.01" iyz="0.0" izz="0.01" />
          </inertial>
       </link>
@@ -216,6 +216,6 @@
          <inertial>
           <origin xyz="0 0 0.043" rpy="0 0 0" />
-            <mass value="0.1" />
-            <inertia ixx="0.1" ixy="0.0" ixz="0.0" iyy="0.1" iyz="0.0" izz="0.1" />
+            <mass value="0.01" />
+            <inertia ixx="0.01" ixy="0.0" ixz="0.0" iyy="0.01" iyz="0.0" izz="0.01" />
          </inertial>
       </link>
@@ -236,6 +236,6 @@
          <inertial>
           <origin xyz = "0 0 0" rpy="0 0 1.57" />
-            <mass value="0.1" />
-            <inertia ixx="0.1" ixy="0.0" ixz="0.0" iyy="0.1" iyz="0.0" izz="0.1" />
+            <mass value="0.01" />
+            <inertia ixx="0.01" ixy="0.0" ixz="0.0" iyy="0.01" iyz="0.0" izz="0.01" />
          </inertial>
       </link>
@@ -258,6 +258,6 @@
          <inertial>
           <origin xyz="0 -0.0007 0" rpy="0 0 1.57" />
-            <mass value="0.1" />
-            <inertia ixx="0.1" ixy="0.0" ixz="0.0" iyy="0.1" iyz="0.0" izz="0.1" />
+            <mass value="0.01" />
+            <inertia ixx="0.01" ixy="0.0" ixz="0.0" iyy="0.01" iyz="0.0" izz="0.01" />
          </inertial>
       </link>
@@ -278,6 +278,6 @@
          <inertial>
           <origin xyz="0 0.0007 0" rpy="0 0 -1.57" />
-            <mass value="0.1" />
-            <inertia ixx="0.1" ixy="0.0" ixz="0.0" iyy="0.1" iyz="0.0" izz="0.1" />
+            <mass value="0.01" />
+            <inertia ixx="0.01" ixy="0.0" ixz="0.0" iyy="0.01" iyz="0.0" izz="0.01" />
          </inertial>
       </link>
@@ -288,5 +288,5 @@
          <child link="shoulder_link" />
          <axis xyz="0 0 1" />
-         <limit lower="-2.617" upper="2.617" effort="0" velocity="0.785" />
+         <limit lower="-3.1415" upper="3.1415" effort="100" velocity="0.785" />
       </joint>
       <joint name="joint_2" type="revolute">
@@ -296,5 +296,5 @@
          <child link="biceps_link" />
          <axis xyz="0 1 0" />
-         <limit lower="-1.571" upper="1.571" effort="0" velocity="1.571" />
+         <limit lower="-1.571" upper="1.571" effort="100" velocity="1.571" />
       </joint>
       <joint name="joint_3" type="revolute">
@@ -303,5 +303,5 @@
          <child link="forearm_link" />
          <axis xyz="0 1 0" />
-         <limit lower="-1.571" upper="1.571" effort="0" velocity="1.571" />
+         <limit lower="-1.571" upper="1.571" effort="100" velocity="1.571" />
       </joint>
       <joint name="joint_4" type="revolute">
@@ -310,5 +310,5 @@
          <child link="wrist_1_link" />
          <axis xyz="0 1 0" />
-         <limit lower="-1.745" upper="1.745" effort="0" velocity="1.571" />
+         <limit lower="-1.745" upper="1.745" effort="100" velocity="1.571" />
       </joint>
       <joint name="joint_5" type="revolute">
@@ -317,5 +317,5 @@
          <child link="wrist_2_link" />
          <axis xyz="0 0 1" />
-         <limit lower="-2.617" upper="2.617" effort="0" velocity="1.571" />
+         <limit lower="-2.617" upper="2.617" effort="100" velocity="1.571" />
       </joint>
       <joint name="joint_6" type="fixed">
@@ -324,5 +324,5 @@
          <child link="gripper_rail_link" />
          <axis xyz="0 0 1" />
-         <limit lower="-0.31" upper="0.1" effort="0" velocity="0.5" />
+         <limit lower="-0.31" upper="0.1" effort="100" velocity="0.5" />
       </joint>
             <joint name="gripper_revolute_joint" type="revolute">
@@ -331,5 +331,5 @@
          <child link="gripper_aux_link" />
          <axis xyz="0 0 1" />
-         <limit lower="0" upper="2.6" effort="0" velocity="0.5" />
+         <limit lower="0" upper="2.6" effort="100" velocity="0.5" />
       </joint>
       <joint name="gripper_prismatic_joint_1" type="prismatic">
@@ -338,5 +338,5 @@
          <child link="gripper_1_link" />
          <axis xyz="0 -1 0" />
-         <limit lower="0" upper="0.027" effort="0" velocity="0.5" />
+         <limit lower="0" upper="0.027" effort="100" velocity="0.5" />
       </joint>
       <joint name="gripper_prismatic_joint_2" type="prismatic">
@@ -346,13 +346,13 @@
          <mimic joint="gripper_prismatic_joint_1" />
          <axis xyz="0 1 0" />
-         <limit lower="0" upper="0.027" effort="0" velocity="0.5" />
+         <limit lower="0" upper="0.027" effort="100" velocity="0.5" />
       </joint>
   <transmission name="tran1">
     <type>transmission_interface/SimpleTransmission</type>
     <joint name="joint_1">
-          <hardwareInterface>hardware_interface/EffortJointInterface</hardwareInterface>
+          <hardwareInterface>hardware_interface/PositionJointInterface</hardwareInterface>
     </joint>
     <actuator name="motor1">
-      <hardwareInterface>hardware_interface/EffortJointInterface</hardwareInterface>
+      <hardwareInterface>hardware_interface/PositionJointInterface</hardwareInterface>
       <mechanicalReduction>1</mechanicalReduction>
     </actuator>
@@ -361,8 +361,8 @@
     <type>transmission_interface/SimpleTransmission</type>
     <joint name="joint_2">
-          <hardwareInterface>hardware_interface/EffortJointInterface</hardwareInterface>
+          <hardwareInterface>hardware_interface/PositionJointInterface</hardwareInterface>
     </joint>
     <actuator name="motor2">
-      <hardwareInterface>hardware_interface/EffortJointInterface</hardwareInterface>
+      <hardwareInterface>hardware_interface/PositionJointInterface</hardwareInterface>
       <mechanicalReduction>1</mechanicalReduction>
     </actuator>
@@ -371,8 +371,8 @@
     <type>transmission_interface/SimpleTransmission</type>
     <joint name="joint_3">
-          <hardwareInterface>hardware_interface/EffortJointInterface</hardwareInterface>
+          <hardwareInterface>hardware_interface/PositionJointInterface</hardwareInterface>
     </joint>
     <actuator name="motor3">
-      <hardwareInterface>hardware_interface/EffortJointInterface</hardwareInterface>
+      <hardwareInterface>hardware_interface/PositionJointInterface</hardwareInterface>
       <mechanicalReduction>1</mechanicalReduction>
     </actuator>
@@ -381,8 +381,8 @@
     <type>transmission_interface/SimpleTransmission</type>
     <joint name="joint_4">
-          <hardwareInterface>hardware_interface/EffortJointInterface</hardwareInterface>
+          <hardwareInterface>hardware_interface/PositionJointInterface</hardwareInterface>
     </joint>
     <actuator name="motor4">
-      <hardwareInterface>hardware_interface/EffortJointInterface</hardwareInterface>
+      <hardwareInterface>hardware_interface/PositionJointInterface</hardwareInterface>
       <mechanicalReduction>1</mechanicalReduction>
     </actuator>
@@ -391,8 +391,8 @@
     <type>transmission_interface/SimpleTransmission</type>
     <joint name="joint_5">
-          <hardwareInterface>hardware_interface/EffortJointInterface</hardwareInterface>
+          <hardwareInterface>hardware_interface/PositionJointInterface</hardwareInterface>
     </joint>
     <actuator name="motor5">
-      <hardwareInterface>hardware_interface/EffortJointInterface</hardwareInterface>
+      <hardwareInterface>hardware_interface/PositionJointInterface</hardwareInterface>
       <mechanicalReduction>1</mechanicalReduction>
     </actuator>
@@ -401,8 +401,8 @@
     <type>transmission_interface/SimpleTransmission</type>
     <joint name="gripper_prismatic_joint_1">
-          <hardwareInterface>hardware_interface/EffortJointInterface</hardwareInterface>
+          <hardwareInterface>hardware_interface/PositionJointInterface</hardwareInterface>
     </joint>
     <actuator name="motor7">
-      <hardwareInterface>hardware_interface/EffortJointInterface</hardwareInterface>
+      <hardwareInterface>hardware_interface/PositionJointInterface</hardwareInterface>
       <mechanicalReduction>1</mechanicalReduction>
     </actuator>
@@ -411,8 +411,8 @@
     <type>transmission_interface/SimpleTransmission</type>
     <joint name="gripper_prismatic_joint_2">
-          <hardwareInterface>hardware_interface/EffortJointInterface</hardwareInterface>
+          <hardwareInterface>hardware_interface/PositionJointInterface</hardwareInterface>
     </joint>
     <actuator name="motor8">
-      <hardwareInterface>hardware_interface/EffortJointInterface</hardwareInterface>
+      <hardwareInterface>hardware_interface/PositionJointInterface</hardwareInterface>
       <mechanicalReduction>1</mechanicalReduction>
     </actuator>

Commit message: Added stability

File: demo_navi/src/urdf/xacro/main.urdf.xacro (robot description, xacro)
@@ -18,10 +18,10 @@
 		<mass value="15"/>
 		<inertia
-			ixx="0.15"
+			ixx="15.0"
 			ixy="0"
 			ixz="0"
-			iyy="0.104167"
+			iyy="15.0"
 			iyz="0"
-			izz="0.254167"
+			izz="9.0"
 		/>
 	</inertial>
@@ -303,5 +303,5 @@
          <child link="shoulder_link" />
          <axis xyz="0 0 1" />
-         <limit lower="-3.1415" upper="3.1415" effort="100" velocity="1.571" />
+         <limit lower="-3.1415" upper="3.1415" effort="100" velocity="1.0" />
       </joint>
       <joint name="joint_2" type="revolute">
@@ -311,5 +311,5 @@
          <child link="biceps_link" />
          <axis xyz="0 1 0" />
-         <limit lower="-1.571" upper="1.571" effort="100" velocity="1.571" />
+         <limit lower="-1.571" upper="1.571" effort="100" velocity="1.0" />
       </joint>
       <joint name="joint_3" type="revolute">
@@ -318,5 +318,5 @@
          <child link="forearm_link" />
          <axis xyz="0 1 0" />
-         <limit lower="-1.571" upper="1.571" effort="100" velocity="1.571" />
+         <limit lower="-1.571" upper="1.571" effort="100" velocity="1.0" />
       </joint>
       <joint name="joint_4" type="revolute">
@@ -325,5 +325,5 @@
          <child link="wrist_1_link" />
          <axis xyz="0 1 0" />
-         <limit lower="-1.745" upper="1.745" effort="100" velocity="1.571" />
+         <limit lower="-1.745" upper="1.745" effort="100" velocity="1.0" />
       </joint>
       <joint name="joint_5" type="revolute">
@@ -332,5 +332,5 @@
          <child link="wrist_2_link" />
          <axis xyz="0 0 1" />
-         <limit lower="-2.617" upper="2.617" effort="100" velocity="1.571" />
+         <limit lower="-2.617" upper="2.617" effort="100" velocity="1.0" />
       </joint>
       <joint name="joint_6" type="fixed">
@@ -346,5 +346,5 @@
          <child link="gripper_aux_link" />
          <axis xyz="0 0 1" />
-         <limit lower="0" upper="2.6" effort="100" velocity="0.5" />
+         <limit lower="0" upper="2.6" effort="10000" velocity="0.5" />
       </joint>
       <joint name="gripper_prismatic_joint_1" type="prismatic">
@@ -353,5 +353,5 @@
          <child link="gripper_1_link" />
          <axis xyz="0 -1 0" />
-         <limit lower="0" upper="0.027" effort="1000" velocity="0.5" />
+         <limit lower="0" upper="0.027" effort="10000" velocity="0.5" />
       </joint>
       <joint name="gripper_prismatic_joint_2" type="prismatic">
@@ -360,5 +360,5 @@
          <child link="gripper_2_link" />
          <axis xyz="0 1 0" />
-         <limit lower="0" upper="0.027" effort="1000" velocity="0.5" />
+         <limit lower="0" upper="0.027" effort="10000" velocity="0.5" />
       </joint>
   <transmission name="tran1">
@@ -567,13 +567,3 @@
     		<material>Gazebo/Black</material>
   	</gazebo>
-  	<gazebo reference="gripper_1_link">
-    		<mu1>5.5</mu1>
-  		<mu2>5.5</mu2>
-		<dampingFactor>10</dampingFactor>
-  	</gazebo>
-  	<gazebo reference="gripper_2_link">
-    		<mu1>5.5</mu1>
-  		<mu2>5.5</mu2>
-  		<dampingFactor>10</dampingFactor>
-  	</gazebo>
 </robot>

Commit message: Updated 1.0

File: demo_navi/src/urdf/xacro/main.urdf.xacro (robot description, xacro)
@@ -11,5 +11,5 @@
   </xacro:sensor_d435>
 	<link name="base_footprint"/>
-  <link name="imu_link"/>
+  	<link name="imu_link"/>
 	<link name="base_link">
 	<inertial>
@@ -51,5 +51,5 @@
 		<child link="base_link" />
 		<origin
-			xyz="0 0 0"
+			xyz="0.144 0 0"
 		/>
 	</joint>
